File: pcb/dnc_v0/dnc.sch (EAGLE design)
At the start: 34 parts, among them IC1 74HC595D, IC2 74HC595D, Q1 200mA/50V, Q2 TSM2306CX, Q3 TSM2306CX, Q4 TSM2306CX, Q6 200mA/50V, U1 ATMEGA168, Y1 16MHZ

Commit message: Reogranise Sch + Add headers
Parts:
- removed JP1: M02-JST-2-PTH-NO_SILK, SparkFun-Connectors:M02-JST-2-PTH-NO_SILK
- removed RANA1, RANA2, RANA3: (no value), SparkFun-Passives:RESISTOR2512
- added C1: 10uF, SparkFun-Passives:CAP_POL6032
- added F1: PTC0603, SparkFun-PowerIC:PTC0603
- added JP10, JP11, JP9: M02JST-PTH-2, SparkFun-Connectors:M02JST-PTH-2
- added JP12: M02-JST-2-PTH-NO_SILK, SparkFun-Connectors:M02-JST-2-PTH-NO_SILK
- added JP2, JP3, JP4: (no value), SparkFun:M03LOCK_LONGPADS
- added JP5, JP6, JP7, JP8: (no value), SparkFun:M02JST-PTH-2
Connections:
- new net N$12: F1.1, JP12.1
- new net OUT_POWER_3: JP11.1
- net 5V: now also JP2.2, JP3.2, JP4.2, U1.AREF
- net ANALOG_IN_1: now also JP2.3; no longer RANA1.2
- net ANALOG_IN_2: now also JP3.3; no longer RANA2.2
- net ANALOG_IN_3: now also JP4.3; no longer RANA3.2
- net GND: now also C1.-, JP10.2, JP11.2, JP12.2, JP2.1, JP3.1, JP4.1, JP9.2; no longer JP1.2, RANA1.1, RANA2.1, RANA3.1
- net IN_1: now also JP5.2
- net IN_2: now also JP6.2
- net IN_3: now also JP7.2
- net IN_4: now also JP8.2
- net OUT_POWER_1: now also JP9.1
- net OUT_POWER_2: now also JP10.1
- net RAW: now also C1.+, F1.2, Q2.D, Q3.D, Q4.D; no longer JP1.1
- net VCC: now also JP5.1, JP6.1, JP7.1, JP8.1; no longer Q2.D, Q3.D, Q4.D, U1.AREF
Other:
- moved on the sheet: IC1, IC2, Q1, Q2, Q3, Q4, Q6, R1, R2, R3, R4, R5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

Commit message: changement de plie de package + liste des composants en stock
Parts:
- removed Y1: 16MHZ, SparkFun-FreqCtrl:RESONATOR16MHZ
- added 8MHZ: RESONATOR, pierre_vv:RESONATOR
- added C16, C7: 0.1uF, rcl:C-EUC0805
- added C2: 10uF, SparkFun:CAP_POL1206
- added ISP1: AVR_SPI_PRG_62X3_LOCK, SparkFun:AVR_SPI_PRG_62X3_LOCK
- added JP13, JP14, JP19: FIDUCIAL1X2.5, SparkFun:FIDUCIAL1X2.5
- added JP15, JP16, JP17, JP18: STAND-OFF, SparkFun:STAND-OFF
- added PROG1: (no value), SparkFun:ARDUINO_SERIAL_PROGRAMLOCK
- added R26: 10K, rcl:R-EU_R0603
- C1: value 10uF -> 0.1uF; device SparkFun-Passives:CAP_POL6032 -> rcl:C-EUC0805
- R1, R2, R4, R5, R6, R7, R8: device SparkFun-Passives:RESISTOR1206 -> SparkFun-Passives:RESISTOR0603-RES
- RCODE, RIN1, RIN2, RIN3, RIN4: device SparkFun-Passives:RESISTOR2512 -> SparkFun-Passives:RESISTOR0603-RES
- renumbered U1 to AT328
Connections:
- removed net /RESET: AT328.PC6(/RESET)
- removed net N$1: AT328.PB7(XTAL2/TOSC2), Y1.3
- removed net N$2: AT328.PB6(XTAL1/TOSC1), Y1.1
- removed net RX: AT328.PD0(RXD)
- removed net TX: AT328.PD1(TXD)
- new net AREF: AT328.AREF, C7.1
- new net DTR: C1.1, PROG1.DTR
- new net N$43: 8MHZ.1, AT328.PB6(XTAL1/TOSC1)
- new net N$44: 8MHZ.3, AT328.PB7(XTAL2/TOSC2)
- new net RESET: AT328.PC6(/RESET), C1.2, ISP1.5, R26.1
- new net RX-I: PROG1.TXO
- new net TX-O: PROG1.RXI
- net 5V: now also AT328.AVCC, AT328.VCC@1, AT328.VCC@2, C16.1, ISP1.2, PROG1.VCC, R26.2; no longer AT328.AREF
- net ACTIVE_ANALOG_RAW: no longer AT328.PD4(XCK/T0)
- net ACTIVE_ANALOG_TEMP: no longer AT328.PD5(T1)
- net ANALOG_IN_1: no longer AT328.PC3(ADC3)
- net ANALOG_IN_2: no longer AT328.PC4(ADC4/SDA)
- net ANALOG_IN_3: no longer AT328.PC5(ADC5/SCL)
- net ANALOG_RAW: no longer AT328.PC1(ADC1)
- net ANALOG_TEMP: no longer AT328.PC2(ADC2)
- net ATMEGA_CS: no longer AT328.PB2(SS/OC1B)
- net CODE: no longer AT328.PC0(ADC0)
- net GND: now also 8MHZ.2, C16.2, C2.-, C7.2, ISP1.6, PROG1.CTS, PROG1.GND; no longer C1.-, Y1.2
- net MISO: now also ISP1.1; no longer AT328.PB4(MISO)
- net MOSI: now also ISP1.4; no longer AT328.PB3(MOSI/OC2)
- net RAW: now also C2.+; no longer C1.+
- net SCK: now also ISP1.3; no longer AT328.PB5(SCK)
- net VCC: no longer AT328.AVCC, AT328.VCC@1, AT328.VCC@2
Other:
- note added: "ATMEGA328P Microcontroler"
- note added: "ISP & PROG connectors"

Commit message: a jour
Parts:
- removed JP12: M02-JST-2-PTH-NO_SILK, SparkFun-Connectors:M02-JST-2-PTH-NO_SILK
- added JP1: M025MM, SparkFun-Connectors:M025MM
- renumbered 8MHZ to 16MHZ
Connections:
- net GND: now also JP1.2; no longer JP12.2
- net N$12: now also JP1.1; no longer JP12.1
Changed lines of the file:
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@@
 <layer number="19" name="Unrouted" color="6" fill="1" visible="yes" active="no"/>
 <layer number="20" name="Dimension" color="15" fill="1" visible="yes" active="no"/>
-<layer number="21" name="tPlace" color="16" fill="1" visible="yes" active="no"/>
-<layer number="22" name="bPlace" color="14" fill="1" visible="yes" active="no"/>
+<layer number="21" name="tPlace" color="7" fill="1" visible="yes" active="no"/>
+<layer number="22" name="bPlace" color="7" fill="1" visible="yes" active="no"/>
 <layer number="23" name="tOrigins" color="15" fill="1" visible="yes" active="no"/>
 <layer number="24" name="bOrigins" color="15" fill="1" visible="yes" active="no"/>
@@
 <part name="F1" library="SparkFun-PowerIC" deviceset="PTC" device="0603"/>
 <part name="GND20" library="SparkFun-Aesthetics" deviceset="GND" device=""/>
-<part name="JP12" library="SparkFun-Connectors" deviceset="M02" device="-JST-2-PTH-NO_SILK"/>
 <part name="GND22" library="SparkFun-Aesthetics" deviceset="GND" device=""/>
 <part name="GND21" library="SparkFun-Aesthetics" deviceset="GND" device=""/>
@@
 <part name="GND36" library="SparkFun" deviceset="GND" device=""/>
 <part name="AT328" library="SparkFun" deviceset="ATMEGA168" device=""/>
-<part name="8MHZ" library="pierre_vv" deviceset="RESONATOR" device=""/>
+<part name="16MHZ" library="pierre_vv" deviceset="RESONATOR" device=""/>
 <part name="U$17" library="SparkFun" deviceset="5V" device=""/>
 <part name="U$18" library="SparkFun" deviceset="5V" device=""/>
@@
 <part name="U$20" library="SparkFun" deviceset="5V" device=""/>
 <part name="U$21" library="SparkFun" deviceset="5V" device=""/>
+<part name="JP1" library="SparkFun-Connectors" deviceset="M02" device="5MM" value="M025MM"/>
 </parts>
 <sheets>
@@
 <instance part="F1" gate="G$1" x="-129.54" y="96.52"/>
 <instance part="GND20" gate="1" x="-116.84" y="71.12"/>
-<instance part="JP12" gate="G$1" x="-160.02" y="96.52" rot="MR180"/>
 <instance part="GND22" gate="1" x="-144.78" y="71.12"/>
 <instance part="GND21" gate="1" x="-96.52" y="71.12" smashed="yes">
@@
 <instance part="GND36" gate="1" x="33.02" y="15.24"/>
 <instance part="AT328" gate="G$1" x="43.18" y="78.74"/>
-<instance part="8MHZ" gate="G$1" x="15.24" y="76.2" rot="R270"/>
+<instance part="16MHZ" gate="G$1" x="15.24" y="76.2" rot="R270"/>
 <instance part="U$17" gate="G$1" x="5.08" y="109.22"/>
 <instance part="U$18" gate="G$1" x="-38.1" y="99.06"/>
@@
 <instance part="U$20" gate="G$1" x="50.8" y="187.96"/>
 <instance part="U$21" gate="G$1" x="38.1" y="154.94"/>
+<instance part="JP1" gate="G$1" x="-160.02" y="96.52" rot="MR180"/>
 </instances>
 <busses>
@@
 </segment>
 <segment>
-<pinref part="JP12" gate="G$1" pin="2"/>
 <wire x1="-152.4" y1="93.98" x2="-144.78" y2="93.98" width="0.1524" layer="91"/>
 <wire x1="-144.78" y1="93.98" x2="-144.78" y2="73.66" width="0.1524" layer="91"/>
 <pinref part="GND22" gate="1" pin="GND"/>
+<pinref part="JP1" gate="G$1" pin="2"/>
 </segment>
 <segment>
@@
 <pinref part="AT328" gate="G$1" pin="GND@2"/>
 <pinref part="AT328" gate="G$1" pin="AGND"/>
-<pinref part="8MHZ" gate="G$1" pin="2"/>
+<pinref part="16MHZ" gate="G$1" pin="2"/>
 </segment>
 <segment>
@@
 <net name="N$12" class="0">
 <segment>
-<pinref part="JP12" gate="G$1" pin="1"/>
 <pinref part="F1" gate="G$1" pin="1"/>
 <wire x1="-152.4" y1="96.52" x2="-134.62" y2="96.52" width="0.1524" layer="91"/>
+<pinref part="JP1" gate="G$1" pin="1"/>
 </segment>
 </net>
@@
 <segment>
 <wire x1="17.78" y1="78.74" x2="20.32" y2="78.74" width="0.1524" layer="91"/>
-<pinref part="8MHZ" gate="G$1" pin="1"/>
+<pinref part="16MHZ" gate="G$1" pin="1"/>
 <pinref part="AT328" gate="G$1" pin="PB6(XTAL1/TOSC1)"/>
 </segment>
@@
 <segment>
 <wire x1="17.78" y1="73.66" x2="20.32" y2="73.66" width="0.1524" layer="91"/>
-<pinref part="8MHZ" gate="G$1" pin="3"/>
+<pinref part="16MHZ" gate="G$1" pin="3"/>
 <pinref part="AT328" gate="G$1" pin="PB7(XTAL2/TOSC2)"/>
 </segment>

Commit message: Reorganize ATmega to work with 5V with tension divider
Parts:
- added RIN5: 10k, SparkFun-Passives:RESISTOR0603-RES
- added RIN6, RIN7: 3.3k, SparkFun-Passives:RESISTOR0603-RES
- JP10, JP11, JP9: value M02JST-PTH-2 -> M025MM; device SparkFun-Connectors:M02JST-PTH-2 -> SparkFun-Connectors:M025MM
- JP5, JP6, JP7, JP8: device SparkFun:M02JST-PTH-2 -> SparkFun:M02LOCK_LONGPADS
- renumbered 16MHZ to 168MHZ
Connections:
- new net MISO_5V: RIN5.2
- new net N$6: RIN6.1, RIN7.2
- net GND: now also RIN7.1
- net MISO: now also RIN5.1, RIN6.2
Changed lines of the file:
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@@
 <part name="GND18" library="SparkFun-Aesthetics" deviceset="GND" device=""/>
 <part name="GND19" library="SparkFun-Aesthetics" deviceset="GND" device=""/>
-<part name="JP5" library="SparkFun" deviceset="M02" device="JST-PTH-2"/>
-<part name="JP6" library="SparkFun" deviceset="M02" device="JST-PTH-2"/>
-<part name="JP7" library="SparkFun" deviceset="M02" device="JST-PTH-2"/>
-<part name="JP8" library="SparkFun" deviceset="M02" device="JST-PTH-2"/>
-<part name="JP9" library="SparkFun-Connectors" deviceset="M02" device="JST-PTH-2"/>
-<part name="JP10" library="SparkFun-Connectors" deviceset="M02" device="JST-PTH-2"/>
-<part name="JP11" library="SparkFun-Connectors" deviceset="M02" device="JST-PTH-2"/>
+<part name="JP5" library="SparkFun" deviceset="M02" device="LOCK_LONGPADS"/>
+<part name="JP6" library="SparkFun" deviceset="M02" device="LOCK_LONGPADS"/>
+<part name="JP7" library="SparkFun" deviceset="M02" device="LOCK_LONGPADS"/>
+<part name="JP8" library="SparkFun" deviceset="M02" device="LOCK_LONGPADS"/>
+<part name="JP9" library="SparkFun-Connectors" deviceset="M02" device="5MM" value="M025MM"/>
+<part name="JP10" library="SparkFun-Connectors" deviceset="M02" device="5MM" value="M025MM"/>
+<part name="JP11" library="SparkFun-Connectors" deviceset="M02" device="5MM" value="M025MM"/>
 <part name="GND9" library="SparkFun-Aesthetics" deviceset="GND" device=""/>
 <part name="GND10" library="SparkFun-Aesthetics" deviceset="GND" device=""/>
@@
 <part name="GND36" library="SparkFun" deviceset="GND" device=""/>
 <part name="AT328" library="SparkFun" deviceset="ATMEGA168" device=""/>
-<part name="16MHZ" library="pierre_vv" deviceset="RESONATOR" device=""/>
-<part name="U$17" library="SparkFun" deviceset="5V" device=""/>
+<part name="168MHZ" library="pierre_vv" deviceset="RESONATOR" device=""/>
+<part name="U$17" library="SparkFun" deviceset="5V" device="" value="5V"/>
 <part name="U$18" library="SparkFun" deviceset="5V" device=""/>
 <part name="U$19" library="SparkFun" deviceset="5V" device=""/>
@@
 <part name="U$21" library="SparkFun" deviceset="5V" device=""/>
 <part name="JP1" library="SparkFun-Connectors" deviceset="M02" device="5MM" value="M025MM"/>
+<part name="RIN5" library="SparkFun-Passives" deviceset="RESISTOR" device="0603-RES" value="10k"/>
+<part name="RIN6" library="SparkFun-Passives" deviceset="RESISTOR" device="0603-RES" value="3.3k"/>
+<part name="RIN7" library="SparkFun-Passives" deviceset="RESISTOR" device="0603-RES" value="3.3k"/>
+<part name="GND2" library="SparkFun-Aesthetics" deviceset="GND" device=""/>
 </parts>
 <sheets>
@@
 <instance part="GND36" gate="1" x="33.02" y="15.24"/>
 <instance part="AT328" gate="G$1" x="43.18" y="78.74"/>
-<instance part="16MHZ" gate="G$1" x="15.24" y="76.2" rot="R270"/>
+<instance part="168MHZ" gate="G$1" x="15.24" y="76.2" rot="R270"/>
 <instance part="U$17" gate="G$1" x="5.08" y="109.22"/>
 <instance part="U$18" gate="G$1" x="-38.1" y="99.06"/>
@@
 <instance part="U$21" gate="G$1" x="38.1" y="154.94"/>
 <instance part="JP1" gate="G$1" x="-160.02" y="96.52" rot="MR180"/>
+<instance part="RIN5" gate="G$1" x="167.64" y="30.48" rot="R90"/>
+<instance part="RIN6" gate="G$1" x="167.64" y="10.16" rot="R90"/>
+<instance part="RIN7" gate="G$1" x="167.64" y="-2.54" rot="R90"/>
+<instance part="GND2" gate="1" x="167.64" y="-12.7"/>
 </instances>
 <busses>
@@
 <pinref part="AT328" gate="G$1" pin="GND@2"/>
 <pinref part="AT328" gate="G$1" pin="AGND"/>
-<pinref part="16MHZ" gate="G$1" pin="2"/>
+<pinref part="168MHZ" gate="G$1" pin="2"/>
 </segment>
 <segment>
@@
 <pinref part="PROG1" gate="G$1" pin="CTS"/>
 </segment>
+<segment>
+<pinref part="RIN7" gate="G$1" pin="1"/>
+<pinref part="GND2" gate="1" pin="GND"/>
+<wire x1="167.64" y1="-7.62" x2="167.64" y2="-10.16" width="0.1524" layer="91"/>
+</segment>
 </net>
 <net name="VCC" class="0">
@@
 <net name="MISO" class="0">
 <segment>
-<wire x1="68.58" y1="48.26" x2="78.74" y2="48.26" width="0.1524" layer="91"/>
-<label x="71.12" y="48.26" size="1.778" layer="95"/>
-</segment>
-<segment>
 <pinref part="U$4" gate="G$1" pin="GPIO9"/>
 <wire x1="58.42" y1="-25.4" x2="45.72" y2="-25.4" width="0.1524" layer="91"/>
@@
 <label x="7.62" y="175.26" size="1.778" layer="95"/>
 <pinref part="ISP1" gate="G$1" pin="1"/>
+</segment>
+<segment>
+<pinref part="RIN5" gate="G$1" pin="1"/>
+<pinref part="RIN6" gate="G$1" pin="2"/>
+<wire x1="167.64" y1="25.4" x2="167.64" y2="20.32" width="0.1524" layer="91"/>
+<wire x1="167.64" y1="20.32" x2="167.64" y2="15.24" width="0.1524" layer="91"/>
+<wire x1="167.64" y1="20.32" x2="182.88" y2="20.32" width="0.1524" layer="91"/>
+<junction x="167.64" y="20.32"/>
+<label x="175.26" y="20.32" size="1.778" layer="95"/>
 </segment>
 </net>
@@
 <wire x1="203.2" y1="121.92" x2="203.2" y2="116.84" width="0.1524" layer="91"/>
 <label x="200.66" y="116.84" size="1.778" layer="95"/>
+</segment>
+<segment>
+<pinref part="C16" gate="G$1" pin="1"/>
+<pinref part="U$19" gate="G$1" pin="5V"/>
+<wire x1="33.02" y1="30.48" x2="33.02" y2="27.94" width="0.1524" layer="91"/>
+</segment>
+<segment>
+<wire x1="50.8" y1="187.96" x2="50.8" y2="175.26" width="0.1524" layer="91"/>
+<wire x1="50.8" y1="175.26" x2="66.04" y2="175.26" width="0.1524" layer="91"/>
+<label x="58.42" y="175.26" size="1.778" layer="95"/>
+<pinref part="PROG1" gate="G$1" pin="VCC"/>
+<pinref part="U$20" gate="G$1" pin="5V"/>
+<pinref part="ISP1" gate="G$1" pin="2"/>
+<wire x1="38.1" y1="175.26" x2="50.8" y2="175.26" width="0.1524" layer="91"/>
+<junction x="50.8" y="175.26"/>
+</segment>
+<segment>
+<pinref part="R26" gate="G$1" pin="2"/>
+<pinref part="U$21" gate="G$1" pin="5V"/>
+<wire x1="38.1" y1="154.94" x2="38.1" y2="152.4" width="0.1524" layer="91"/>
 </segment>
 <segment>
@@
 <wire x1="5.08" y1="99.06" x2="5.08" y2="109.22" width="0.1524" layer="91"/>
 <pinref part="U$17" gate="G$1" pin="5V"/>
-</segment>
-<segment>
-<pinref part="C16" gate="G$1" pin="1"/>
-<pinref part="U$19" gate="G$1" pin="5V"/>
-<wire x1="33.02" y1="30.48" x2="33.02" y2="27.94" width="0.1524" layer="91"/>
-</segment>
-<segment>
-<wire x1="50.8" y1="187.96" x2="50.8" y2="175.26" width="0.1524" layer="91"/>
-<wire x1="50.8" y1="175.26" x2="66.04" y2="175.26" width="0.1524" layer="91"/>
-<label x="58.42" y="175.26" size="1.778" layer="95"/>
-<pinref part="PROG1" gate="G$1" pin="VCC"/>
-<pinref part="U$20" gate="G$1" pin="5V"/>
-<pinref part="ISP1" gate="G$1" pin="2"/>
-<wire x1="38.1" y1="175.26" x2="50.8" y2="175.26" width="0.1524" layer="91"/>
-<junction x="50.8" y="175.26"/>
-</segment>
-<segment>
-<pinref part="R26" gate="G$1" pin="2"/>
-<pinref part="U$21" gate="G$1" pin="5V"/>
-<wire x1="38.1" y1="154.94" x2="38.1" y2="152.4" width="0.1524" layer="91"/>
 </segment>
 </net>
@@
 <segment>
 <wire x1="17.78" y1="78.74" x2="20.32" y2="78.74" width="0.1524" layer="91"/>
-<pinref part="16MHZ" gate="G$1" pin="1"/>
+<pinref part="168MHZ" gate="G$1" pin="1"/>
 <pinref part="AT328" gate="G$1" pin="PB6(XTAL1/TOSC1)"/>
 </segment>
@@
 <segment>
 <wire x1="17.78" y1="73.66" x2="20.32" y2="73.66" width="0.1524" layer="91"/>
-<pinref part="16MHZ" gate="G$1" pin="3"/>
+<pinref part="168MHZ" gate="G$1" pin="3"/>
 <pinref part="AT328" gate="G$1" pin="PB7(XTAL2/TOSC2)"/>
 </segment>
 </net>
+<net name="MISO_5V" class="0">
+<segment>
+<wire x1="147.32" y1="43.18" x2="167.64" y2="43.18" width="0.1524" layer="91"/>
+<pinref part="RIN5" gate="G$1" pin="2"/>
+<wire x1="167.64" y1="43.18" x2="167.64" y2="35.56" width="0.1524" layer="91"/>
+<label x="149.86" y="43.18" size="1.778" layer="95"/>
+</segment>
+<segment>
+<wire x1="68.58" y1="48.26" x2="78.74" y2="48.26" width="0.1524" layer="91"/>
+<label x="71.12" y="48.26" size="1.778" layer="95"/>
+</segment>
+</net>
+<net name="N$6" class="0">
+<segment>
+<pinref part="RIN6" gate="G$1" pin="1"/>
+<pinref part="RIN7" gate="G$1" pin="2"/>
+<wire x1="167.64" y1="5.08" x2="167.64" y2="2.54" width="0.1524" layer="91"/>
+</segment>
+</net>
