File: pcb/dnc_v1/dnc.brd (EAGLE design)
At the start: 98.7 x 83.2 mm, 66 parts, among them Q5 TSM2306CX, Q7 TSM2306CX, Q8 TSM2306CX

Commit message: avance sur v1
Parts:
- removed 3.3/5: (no value), SparkFun:1X02_LONGPADS
- removed EXT5, EXT6: EXT-DNC, pierre_vv:EXTPINDNC
- removed MOS_TEMP: 200mA/50V, SparkFun-DiscreteSemi:SOT23-3
- removed PTC: (no value), ptc-ntc:P679
- removed REG1, REG2: 74HC595D, 74xx-eu:SO16
- removed RTEMP0: 100k, SparkFun-Passives:0603-RES
- removed RTEMP2: (no value), SparkFun-Passives:0603-RES
- removed U$5: DC/DC_SEED, pierre_vv:DC/DC_SEED
- added C1: (no value), rcl:PANASONIC_E
- added C3, C4: 0.1uF, rcl:C0603
- added C5, C6: 1uF, rcl:C0603
- added D1: 40v5A, diode:SMC
- added D2: 1.8v, SparkFun-DiscreteSemi:SOD-123
- added D3: 33v, SparkFun-DiscreteSemi:SOD-123
- added IC1: LM2596S, national-semiconductor:TO263-5
- added L1: 100nH, SparkFun:CDRH125
- added Q1: IRF9321PBF, pierre_vv:SO-8
- added RBAT3: 100K, SparkFun-Passives:0603-RES
- added U1: AP2202-ADJ, SparkFun-PowerIC:SOT23-5
- added U2: 74HCT595D, IC:SO16
- added U3, U4: 74LVC1G08SE-7, SparkFun-DigitalIC:SOT353
- C2: value 10uF -> 680uF30mm; device SparkFun:EIA3216 -> SparkFun:CPOL-RADIAL-1000UF-25V
- F1: value PTCPTH -> 8A; device SparkFun-PowerIC:PTC -> SparkFun:PTC
- RBAT1: value 100k -> 100k1%
- RBAT2: value 10k -> 10k1%
- moved F1 217.8 mm to (-70.0, -85.0), turned to 0 degrees
Connections:
- removed net ACTIVE_ANALOG_TEMP: MOS_TEMP.1, RTEMP0.1
- removed net N$10: EXT5.FREE
- removed net N$11: MOS_TEMP.3, PTC.2
- removed net N$12: F1.P$1, RAW_IN.1
- removed net N$7: REG1.9, REG2.14
- removed net N$9: EXT6.FREE
- removed net RAW: C2.A, EXT1.RAW, EXT2.RAW, EXT3.RAW, EXT4.RAW, EXT5.RAW, EXT6.RAW, F1.P$2, MOS_PWR1.3, MOS_PWR2.3, MOS_PWR3.3, RBAT1.2, U$5.IN+
- removed net RST10: REG2.1
- removed net RST11: REG2.2
- removed net RST12: REG2.3
- removed net RST13: REG2.4
- removed net RST14: REG2.5
- removed net RST15: REG2.6
- removed net RST16: REG2.7
- removed net RST9: REG2.15
- removed net VCC: REG1.16, REG2.16
- new net MOSI_5V: TITREUR1.7, TITREUR2.7, U4.4
- new net N$1: D1.C, IC1.2, L1.1
- new net PROTECT_GATE: D2.A, Q1.4, RBAT3.1
- new net RAW_FUSED: C2.1, C3.1, EXT1.RAW, EXT2.RAW, EXT3.RAW, EXT4.RAW, F1.P$2, IC1.1, MOS_PWR1.3, MOS_PWR2.3, MOS_PWR3.3, RBAT1.2
- new net RAW_POL_PROTECTED: D2.C, D3.C, F1.P$1MOV, Q1.1, Q1.2, Q1.3
- new net RAW_UNPROTECTED: Q1.5, Q1.6, Q1.7, Q1.8, RAW_IN.1
- new net SCK_TITREUR: TITREUR1.5, TITREUR2.5, U3.4
- net +3V3: now also C6.1, U1.5; no longer 3.3/5.1, EXT5.3.3V, EXT6.3.3V
- net +5V: now also C1.+, C4.1, C5.1, IC1.4, L1.2, U1.1, U1.3, U2.10, U2.16, U3.5, U4.1, U4.5; no longer 3.3/5.2, EXT5.5V, EXT6.5V, PTC.1, U$5.OUT+
- net /CS_EXT_5: no longer EXT5./RESET
- net /CS_EXT_6: no longer EXT6./RESET
- net ANALOG_TEMP: no longer MOS_TEMP.2, RTEMP2.1
- net CODE: no longer EXT5.RETOURANALOG, EXT6.RETOURANALOG
- net GND: now also C1.-, C2.2, C3.2, C4.2, C5.2, C6.2, D1.A, D3.A, IC1.3, IC1.5, RBAT3.2, U1.2, U2.13, U2.8, U3.3, U4.3; no longer C2.C, EXT5.1_GND, EXT6.1_GND, REG1.13, REG1.8, REG2.13, REG2.8, RTEMP0.2, RTEMP2.2, U$5.IN-, U$5.OUT-
- net MISO: no longer EXT5.MISO, EXT6.MISO
- net MOSI: now also U4.2; no longer EXT5.MOSI, EXT6.MOSI, REG1.14, TITREUR1.7, TITREUR2.7
- net REG_CLR: no longer REG1.10, REG2.10
- net REG_RCK: now also U3.1; no longer REG1.12, REG2.12
- net RST1: now also U2.15; no longer REG1.15
- net RST2: now also U2.1; no longer REG1.1
- net RST3: now also U2.2; no longer REG1.2
- net RST4: now also U2.3; no longer REG1.3
- net RST5: now also U2.4; no longer REG1.4
- net RST6: now also U2.5; no longer REG1.5
- net RST7: now also U2.6; no longer REG1.6
- net RST8: now also U2.7; no longer REG1.7
- net SCK: now also U2.11, U3.2; no longer EXT5.SCK, EXT6.SCK, REG1.11, REG2.11, TITREUR1.5, TITREUR2.5
Routing:
- net +3V3: track 403.0 -> 0.00 mm, vias 7 -> 0
- net SCK: track 344.6 -> 0.00 mm, vias 11 -> 0
- net MOSI: track 342.0 -> 0.00 mm, vias 9 -> 0
- net MISO: track 329.7 -> 0.00 mm, vias 9 -> 0
- net RAW: track 272.6 -> 0.00 mm, vias 7 -> 0
- net +5V: track 250.7 -> 0.00 mm, vias 7 -> 0
- net CODE: track 170.9 -> 0.00 mm, vias 3 -> 0
- net RESET: track 122.1 -> 0.00 mm, vias 1 -> 0
- net /CS_EXT_6: track 71.2 -> 0.00 mm, vias 2 -> 0
- net /CS_EXT_1: track 69.8 -> 0.00 mm, vias 2 -> 0
- net /CS_EXT_5: track 56.2 -> 0.00 mm, vias 3 -> 0
- net /CS_EXT_3: track 55.3 -> 0.00 mm, vias 2 -> 0
- net ACTIVE_OUT_POWER_3: track 49.9 -> 0.00 mm, vias 2 -> 0
- net /CS_EXT_4: track 43.6 -> 0.00 mm, vias 2 -> 0
- net /CS_EXT_2: track 42.2 -> 0.00 mm, vias 1 -> 0
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
Commit message: in progress
Parts:
- removed 8MHZ: RESONATOR, pierre_vv:RESONATOR_7MM
- removed A_IN1, A_IN2, A_IN3: DNC_IN3, pierre_vv:DNC_IN3
- removed IN1, IN2, IN3, IN4, OUT1, OUT2, OUT3: DNC_IN2, pierre_vv:DNC_IN2
- removed MOS_PWR1, MOS_PWR2, MOS_PWR3, Q5, Q7, Q8: TSM2306CX, SparkFun-DiscreteSemi:SOT323
- removed PWR_OUT1, PWR_OUT2, PWR_OUT3: DNC_IN2PWR, pierre_vv:DNC_IN2_PWR
- removed RIN1, RIN2, RIN3, RIN4: (no value), SparkFun-Passives:0603-RES
- removed RIN10, RIN8, RIN9, ROUT1, ROUT2, ROUT3: 100k, SparkFun-Passives:0603-RES
- added 16MHZ: 16MHZ, SparkFun-FreqCtrl:RESONATOR-SMD
- added C10, C8: 1uF, rcl:C0603
- added C7, C9: 0.1uF, rcl:C0603
- added D4, D5: 40v5A, diode:SMC
- added IC2: 74S244DW, 74xx-us:SO20W
- added L2, L3: 100nH, SparkFun:CDRH125
- added PLUG_3.81_1: FLEX, pierre_vv:PLUG_03
- added PLUG_3.81_2_1: LED10W2, pierre_vv:PLUG_02
- added PLUG_3.81_2_2: LED10W1, pierre_vv:PLUG_02
- added PLUG_3.81_6_1: M06, pierre_vv:PLUG_06
- added Q10, Q11, Q2, Q4, Q6, Q9: BSS670, SparkFun-DiscreteSemi:SOT23-3
- added Q3: BSS138, SparkFun-DiscreteSemi:SOT23-3
- added RBAT10, RBAT11, RBAT12, RBAT13, RBAT16, RBAT17, RBAT18, RBAT19, RBAT20, RBAT21, RBAT4, RBAT5, RBAT8, RBAT9: 100K, SparkFun-Passives:0603-RES
- added RBAT14, RBAT15: 0.110, SparkFun-Passives:0603-RES
- added RBAT22, RBAT23, RBAT24, RBAT25, RBAT6, RBAT7: 10K, SparkFun-Passives:0603-RES
- added SJ1, SJ2: JUMPER-PTH-2-NC, SparkFun-Passives:PTH-JUMPER-NC_BOTTOM_NO_SILK
- added U5: AL8807, SparkFun-PowerIC:SOT23-5
- AT328: value ATMEGA168 -> ATMEGA328
- MOS_BAT: value 200mA/50V -> MOSFET-NCHANNELBSS138
- U3: value 74LVC1G08SE-7 -> TC7SU04F; device SparkFun-DigitalIC:SOT353 -> SparkFun-DigitalIC:SOT23-5
- U4: value 74LVC1G08SE-7 -> AL8807; device SparkFun-DigitalIC:SOT353 -> SparkFun-PowerIC:SOT23-5
- moved U4 105.8 mm to (-118.0, -206.0)
- moved U3 98.1 mm to (-114.0, -193.0)
Connections:
- net REG_CLR renamed LED_R
- removed net /CS_EXT_5: U$4.3
- removed net /CS_EXT_6: U$4.6
- removed net ACTIVE_OUT_1: Q5.1, RIN8.2, U$4.36
- removed net ACTIVE_OUT_2: Q7.1, RIN9.2, U$4.38
- removed net ACTIVE_OUT_3: Q8.1, RIN10.2, U$4.40
- removed net ACTIVE_OUT_POWER_1: AT328.32, MOS_PWR1.1, ROUT1.2
- removed net ACTIVE_OUT_POWER_2: AT328.1, MOS_PWR2.1, ROUT2.2
- removed net ACTIVE_OUT_POWER_3: AT328.10, MOS_PWR3.1, ROUT3.2
- removed net ANALOG_IN_1: AT328.26, A_IN1.3
- removed net ANALOG_IN_2: AT328.27, A_IN2.3
- removed net ANALOG_IN_3: AT328.28, A_IN3.3
- removed net ANALOG_TEMP: AT328.25
- removed net IN_1: IN1.2, RIN1.2, U$4.37
- removed net IN_2: IN2.2, RIN2.2, U$4.35
- removed net IN_3: IN3.2, RIN3.2, U$4.33
- removed net IN_4: IN4.2, RIN4.2, U$4.31
- removed net OUT_1: OUT1.1, Q5.2
- removed net OUT_2: OUT2.1, Q7.2
- removed net OUT_3: OUT3.1, Q8.2
- removed net OUT_POWER_1: MOS_PWR1.2, PWR_OUT1.1
- removed net OUT_POWER_2: MOS_PWR2.2, PWR_OUT2.1
- removed net OUT_POWER_3: MOS_PWR3.2, PWR_OUT3.1
- removed net SCK_TITREUR: TITREUR1.5, TITREUR2.5, U3.4
- new net ALL_CS_ENABLE_ACTIVE_LOW: IC2.1, IC2.19, U2.13, U3.4
- new net ATMEGA_CS_5V: AT328.14, IC2.5
- new net CS_TRIGGER_ACTIVE_HIGH: U$4.37, U3.2
- new net EXT1_CS: IC2.2, U$4.3
- new net EXT1_CS_5V: IC2.18
- new net EXT2_CS: IC2.4, U$4.5
- new net EXT2_CS_5V: IC2.16
- new net EXT3_CS: IC2.6, U$4.7
- new net EXT3_CS_5V: IC2.14
- new net EXT4_CS: IC2.13, IC2.7, U$4.29
- new net EXT5_CS: U$4.31
- new net GYRO_1: AT328.25, Q4.1, RBAT16.2
- new net GYRO_2: AT328.26, Q2.1, RBAT17.2
- new net GYRO_3: AT328.27, Q6.1, RBAT18.2
- new net GYRO_4: AT328.28, Q9.1, RBAT19.2
- new net INT_ATMEGA: RBAT22.1, RBAT23.2, U$4.38
- new net INT_ATMEGA_5V: AT328.2, RBAT22.2
- new net INT_TELECO: RBAT24.1, RBAT25.2, U$4.40
- new net INT_TELECO_5V: RBAT24.2
- new net LED+1: C8.1, PLUG_3.81_2_1.1, RBAT14.1, SJ1.2, U4.4
- new net LED+2: C10.1, PLUG_3.81_2_2.1, RBAT15.1, SJ2.2, U5.4
- new net LED-1: C8.2, L2.2, PLUG_3.81_2_1.2
- new net LED-2: C10.2, L3.2, PLUG_3.81_2_2.2
- new net LED_G: U$4.15
- new net MISO_5V: AT328.16, ISP.1, Q3.3, RBAT7.1
- new net N$10: PLUG_3.81_6_1.2, Q4.3
- new net N$11: PLUG_3.81_6_1.3, Q2.3
- new net N$12: PLUG_3.81_6_1.4, Q6.3
- new net N$13: PLUG_3.81_6_1.5, Q9.3
- new net N$14: PLUG_3.81_1.2, Q10.3
- new net N$15: EXT1.5V, EXT2.5V, EXT3.5V, EXT4.5V
- new net N$16: AT328.32
- new net N$6: D4.A, L2.1, U4.1
- new net N$7: D5.A, L3.1, U5.1
- new net N$9: PLUG_3.81_1.3, Q11.3
- new net PWM_FLEX_1: AT328.1, Q10.1, RBAT20.2
- new net PWM_FLEX_2: AT328.13, Q11.1, RBAT21.2
- new net PWM_LED_1: AT328.9, U5.3
- new net PWM_LED_2: AT328.10, U4.3
- new net RESET_5V: AT328.29, ISP.5
- new net SCK_5V: AT328.17, IC2.9, ISP.3, TITREUR1.5, TITREUR2.5
- new net TELECO_CS: IC2.17, U$4.35
- new net TELECO_CS_5V: IC2.3
- net +3V3: now also Q3.1, RBAT6.2; no longer AT328.18, AT328.4, AT328.6, A_IN1.2, A_IN2.2, A_IN3.2, C3.3.1, IN1.1, IN2.1, IN3.1, IN4.1, ISP.2, PROG1.4, RRST.2
- net +5V: now also AT328.18, AT328.4, AT328.6, C3.3.1, IC2.20, ISP.2, PROG1.4, RBAT10.2, RBAT11.2, RBAT12.2, RBAT13.2, RBAT4.2, RBAT5.2, RBAT7.2, RBAT8.2, RBAT9.2, RRST.2; no longer EXT1.5V, EXT2.5V, EXT3.5V, EXT4.5V, Q5.3, Q7.3, Q8.3, U4.1, U4.5
- net /CS_EXT_1: no longer U$4.32
- net /CS_EXT_2: no longer U$4.29
- net /CS_EXT_3: no longer U$4.7
- net /CS_EXT_4: no longer U$4.5
- net ACTIVE_ANALOG_RAW: no longer AT328.2
- net ATMEGA_CS: now also IC2.15, U$4.33; no longer AT328.14, U$4.16
- net GND: now also 16MHZ.2, C7.2, C9.2, IC2.10, Q10.2, Q11.2, Q2.2, Q4.2, Q6.2, Q9.2, RBAT16.1, RBAT17.1, RBAT18.1, RBAT19.1, RBAT20.1, RBAT21.1, RBAT23.1, RBAT25.1, U$4.6, U4.2, U5.2; no longer 8MHZ.2, A_IN1.1, A_IN2.1, A_IN3.1, OUT1.2, OUT2.2, OUT3.2, PWR_OUT1.2, PWR_OUT2.2, PWR_OUT3.2, RIN1.1, RIN10.1, RIN2.1, RIN3.1, RIN4.1, RIN8.1, RIN9.1, ROUT1.1, ROUT2.1, ROUT3.1, U2.13, U4.3
- net MISO: now also Q3.2, RBAT6.1; no longer AT328.16, ISP.1
- net MOSI: now also IC2.8; no longer AT328.15, ISP.4, U4.2
- net MOSI_5V: now also AT328.15, IC2.12, ISP.4; no longer U4.4
- net N$43: now also 16MHZ.1; no longer 8MHZ.1
- net N$44: now also 16MHZ.3; no longer 8MHZ.3
- net RAW_FUSED: now also C7.1, C9.1, D4.C, D5.C, PLUG_3.81_1.1, PLUG_3.81_6_1.1, PLUG_3.81_6_1.6, RBAT14.2, RBAT15.2, SJ1.1, SJ2.1, U4.5, U5.5; no longer MOS_PWR1.3, MOS_PWR2.3, MOS_PWR3.3
- net REG_RCK: no longer U3.1
- net RESET: no longer AT328.29, ISP.5
- net RST1: now also RBAT4.1
- net RST2: now also RBAT5.1
- net RST3: now also RBAT8.1
- net RST4: now also RBAT9.1
- net RST5: now also RBAT10.1
- net RST6: now also RBAT11.1
- net RST7: now also RBAT12.1
- net RST8: now also RBAT13.1
- net SCK: now also IC2.11; no longer AT328.17, ISP.3, U3.2

Commit message: in progress 2
Parts:
- removed EXT1, EXT2, EXT3, EXT4: EXT-DNC, pierre_vv:EXTPINDNC
- added U$1: EXT1, pierre_vv:EXTPINDNC
- added U$2: EXT2, pierre_vv:EXTPINDNC
- added U$3: EXT3, pierre_vv:EXTPINDNC
- added U$5: EXT4, pierre_vv:EXTPINDNC
- added U$8: RJ45-EXTDNC, con-amphenol-rj45-ld:RJ45-TRAFO
- C3.3, CMHZ, CRST: device rcl:C0805 -> rcl:C0603
- RBAT23, RBAT25: value 10K -> 20K
Connections:
- removed net /CS_EXT_1: EXT1./RESET
- removed net /CS_EXT_2: EXT2./RESET
- removed net /CS_EXT_3: EXT3./RESET
- removed net /CS_EXT_4: EXT4./RESET
- removed net N$15: EXT1.5V, EXT2.5V, EXT3.5V, EXT4.5V
- removed net N$21: EXT1.FREE
- removed net N$4: EXT2.FREE
- removed net N$5: EXT3.FREE
- removed net N$8: EXT4.FREE
- new net EXT4_CS_5V: U$5./CS
- net +3V3: no longer EXT1.3.3V, EXT2.3.3V, EXT3.3.3V, EXT4.3.3V
- net +5V: now also U$1.5V, U$2.5V, U$3.5V, U$5.5V, U$8.7
- net CODE: now also U$1.RETOURANALOG, U$2.RETOURANALOG, U$3.RETOURANALOG, U$5.RETOURANALOG, U$8.5; no longer EXT1.RETOURANALOG, EXT2.RETOURANALOG, EXT3.RETOURANALOG, EXT4.RETOURANALOG
- net EXT1_CS_5V: now also U$1./CS
- net EXT2_CS_5V: now also U$2./CS
- net EXT3_CS_5V: now also U$3./CS
- net GND: now also U$1.1_GND, U$1.GND2, U$2.1_GND, U$2.GND2, U$3.1_GND, U$3.GND2, U$5.1_GND, U$5.GND2, U$8.8; no longer EXT1.1_GND, EXT2.1_GND, EXT3.1_GND, EXT4.1_GND
- net INT_TELECO_5V: now also U$8.6
- net MISO: no longer EXT1.MISO, EXT2.MISO, EXT3.MISO, EXT4.MISO
- net MISO_5V: now also U$1.MISO, U$2.MISO, U$3.MISO, U$5.MISO, U$8.1
- net MOSI: no longer EXT1.MOSI, EXT2.MOSI, EXT3.MOSI, EXT4.MOSI
- net MOSI_5V: now also U$1.MOSI, U$2.MOSI, U$3.MOSI, U$5.MOSI, U$8.2
- net RAW_FUSED: now also U$1.RAW, U$1.RAW2, U$2.RAW, U$2.RAW2, U$3.RAW, U$3.RAW2, U$5.RAW, U$5.RAW2; no longer EXT1.RAW, EXT2.RAW, EXT3.RAW, EXT4.RAW
- net SCK: no longer EXT1.SCK, EXT2.SCK, EXT3.SCK, EXT4.SCK, U2.11
- net SCK_5V: now also U$1.SCK, U$2.SCK, U$3.SCK, U$5.SCK, U$8.3, U2.11
- net TELECO_CS_5V: now also U$8.4

Commit message: schematic fini début routage
Parts:
- removed C5, C6: 1uF, rcl:C0603
- removed MOS_BAT: MOSFET-NCHANNELBSS138, SparkFun-DiscreteSemi:SOT23-3
- removed U1: AP2202-ADJ, SparkFun-PowerIC:SOT23-5
- added C11, C12, C13: 1uF, rcl:C0603
- added C3.1: 0.1uF, rcl:C0603
- added D6: (no value), SparkFun-DiscreteSemi:SMA-DIODE_ALT
- added K1: G5L, relay:G5LE
- added LEDG, LEDR: (no value), led:CHIPLED_0603
- added PLUG_3.81_2: FLEX, pierre_vv:PLUG_03
- added Q12, Q5, Q7, Q8: BSS138, SparkFun-DiscreteSemi:SOT23-3
- added RBAT26, RBAT27, RBAT29: 100K, SparkFun-Passives:0603-RES
- added RBAT28, RBAT30: 220, SparkFun-Passives:0603-RES
- added RBAT31, RBAT32, RBAT35: 56K, SparkFun-Passives:0603-RES
- added RBAT33, RBAT34, RBAT36: 33K, SparkFun-Passives:0603-RES
- added RBAT37: 1K, SparkFun-Passives:0603-RES
- added S1: (no value), switch-omron:B3F-31XX
- added U$6: M08, pierre_vv:PLUG_08
- Q10, Q11: value BSS670 -> BSS316
- moved PLUG_3.81_1 466.9 mm to (43.2, 80.0)
- moved U$3 450.2 mm to (12.7, 49.3), turned to 90 degrees
- moved U$5 447.2 mm to (13.3, 39.8), turned to 90 degrees
- moved PLUG_3.81_6_1 444.8 mm to (64.8, 80.0)
- moved U$2 429.9 mm to (12.7, 30.2), turned to 90 degrees
- moved PLUG_3.81_2_2 414.6 mm to (92.7, 80.0)
- moved U$1 409.7 mm to (12.7, 11.2), turned to 90 degrees
- moved PLUG_3.81_2_1 390.8 mm to (82.5, 80.0)
- moved IC2 271.1 mm to (40.6, 26.1), turned to 180 degrees
- moved F1 177.8 mm to (6.35, 75.6), turned to 270 degrees
- moved D3 163.4 mm to (9.53, 79.1), turned to 270 degrees
- moved Q1 161.3 mm to (21.0, 79.4)
- moved RBAT3 156.5 mm to (12.4, 78.1), turned to 90 degrees
- moved D2 154.6 mm to (15.0, 79.1), turned to 270 degrees
- moved U2 151.9 mm to (25.7, 21.9), turned to 180 degrees
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Connections:
- removed net N$16: AT328.32
- removed net RESET_5V: AT328.29, ISP.5
- new net FLOAT1: AT328.19, U$6.2
- new net FLOAT2: AT328.22, U$6.3
- new net LEDG: Q12.1, RBAT29.2
- new net LEDR: LEDG.C, LEDR.C, Q12.3, Q8.1, Q8.3, RBAT27.2
- new net N$15: K1.O, PLUG_3.81_2.1
- new net N$17: K1.S, PLUG_3.81_2.3
- new net N$18: LEDG.A, RBAT30.1
- new net N$19: U$4.22
- new net N$20: RBAT32.1, RBAT34.1, U$6.6
- new net N$21: LEDR.A, RBAT28.1
- new net N$22: RBAT31.1, RBAT33.1, S1.2, U$6.7
- new net N$23: RBAT35.1, RBAT36.1, U$6.5
- new net N$25: RBAT37.1, U$6.1
- new net N$4: U2.10
- new net N$5: D6.A, K1.2, Q5.3
- new net N$8: K1.P, PLUG_3.81_2.2
- new net PUSH1: AT328.32, C13.1, RBAT33.2
- new net PUSH2: AT328.11, C12.1, RBAT34.2
- new net PUSH3: AT328.12, C11.1, RBAT36.2
- new net RELAY1: Q5.1, RBAT26.2, U$4.12
- net +3V3: no longer C6.1, U$4.18, U1.5
- net +5V: now also C3.1.1, D6.C, K1.1, RBAT28.2, RBAT30.2, RBAT31.2, RBAT32.2, RBAT35.2, RBAT37.2; no longer C5.1, U1.1, U1.3, U2.10
- net ACTIVE_ANALOG_RAW: now also Q7.1; no longer MOS_BAT.1
- net ANALOG_RAW: now also Q7.2; no longer MOS_BAT.2
- net EXT1_CS: now also IC2.8; no longer IC2.2
- net EXT1_CS_5V: now also IC2.12; no longer IC2.18
- net EXT2_CS: now also IC2.6; no longer IC2.4
- net EXT2_CS_5V: now also IC2.14; no longer IC2.16
- net EXT3_CS: now also IC2.4; no longer IC2.6
- net EXT3_CS_5V: now also IC2.16; no longer IC2.14
- net GND: now also C11.2, C12.2, C13.2, C3.1.2, Q12.2, Q5.2, Q8.2, RBAT26.1, RBAT27.1, RBAT29.1, S1.1, U$6.4, U$6.8; no longer C5.2, C6.2, U1.2
- net LED_G: now also U$4.18
- net LED_R: now also U$4.16
- net MOSI: now also IC2.2; no longer IC2.8
- net MOSI_5V: now also IC2.18, U2.14; no longer IC2.12
- net N$3: now also Q7.3; no longer MOS_BAT.3
- net REG_RCK: now also U2.12
- net RESET: now also AT328.29, ISP.5
Routing:
- net RAW_FUSED: track 0.00 -> 114.6 mm
- net +5V: track 0.00 -> 32.4 mm
- net N$1: track 0.00 -> 26.9 mm
- net RAW_POL_PROTECTED: track 0.00 -> 13.4 mm
- net RAW_UNPROTECTED: track 0.00 -> 9.58 mm
- net PROTECT_GATE: track 0.00 -> 5.92 mm
- removed copper zone on layer 1, net GND
- removed copper zone on layer 16, net GND
Other:
- board size 98.7 x 83.2 mm -> 99 x 87 mm

Commit message: routage terminé
Parts:
- removed U$3: EXT3, pierre_vv:EXTPINDNC
- removed U$5: EXT4, pierre_vv:EXTPINDNC
- added C3.2: 0.1uF, rcl:C0603
- added JP1: M05X2SHD_LOCK, SparkFun:2X5-SHROUDED_LOCK
- added RBAT38, RBAT39: 10K, SparkFun-Passives:0603-RES
- PLUG_3.81_2: value FLEX -> RELAY
- SJ1, SJ2: value JUMPER-PTH-2-NC -> JUMPER-PTH-2-NO; device SparkFun-Passives:PTH-JUMPER-NC_BOTTOM_NO_SILK -> SparkFun-Passives:PTH-JUMPER-2-NO_NO_SILK
- moved C3.1 590.3 mm to (41.7, 14.7), turned to 270 degrees
- moved C13 580.8 mm to (10.8, 34.9), turned to 180 degrees
- moved RBAT29 573.5 mm to (49.5, 60.3)
- moved C12 572.3 mm to (10.8, 29.2), turned to 180 degrees
- moved S1 571.1 mm to (3.92, 49.2), turned to 270 degrees
- moved Q12 568.3 mm to (49.5, 62.9), turned to 90 degrees
- moved RBAT37 564.2 mm to (11.4, 9.53), turned to 270 degrees
- moved C11 563.8 mm to (10.8, 23.5), turned to 180 degrees
- moved RBAT27 557.3 mm to (49.5, 55.2)
- moved Q8 556.9 mm to (49.5, 57.8), turned to 90 degrees
- moved RBAT36 555.4 mm to (10.8, 25.4)
- moved RBAT34 555.2 mm to (10.8, 31.1)
- moved RBAT33 555.0 mm to (10.8, 36.8)
- moved RBAT35 554.5 mm to (10.8, 27.3)
- moved RBAT32 554.3 mm to (10.8, 33.0)
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Connections:
- net ALL_CS_ENABLE_ACTIVE_LOW renamed ALL_CS_ENABLE_ACTIVE_LOW_5V
- removed net ACTIVE_ANALOG_RAW: Q7.1, RBAT0.2
- removed net EXT4_CS: IC2.13, IC2.7, U$4.29
- removed net EXT4_CS_5V: U$5./CS
- removed net EXT5_CS: U$4.31
- removed net N$17: K1.S, PLUG_3.81_2.3
- removed net N$19: U$4.22
- removed net N$5: D6.A, K1.2, Q5.3
- new net N$16: D6.A, K1.1, Q5.3
- new net READ_BATTERY: Q7.1, RBAT0.2, U$4.22
- new net REG_RCK_5V: IC2.18, U2.12
- net +5V: now also C3.2.1, K1.2, U2.10; no longer K1.1, U$3.5V, U$5.5V
- net ATMEGA_CS: now also IC2.13; no longer IC2.15
- net ATMEGA_CS_5V: now also IC2.7; no longer IC2.5
- net CODE: no longer U$3.RETOURANALOG, U$5.RETOURANALOG
- net CS_TRIGGER_ACTIVE_HIGH: now also RBAT38.2, U$4.29; no longer U$4.37
- net EXT3_CS_5V: no longer U$3./CS
- net GND: now also C3.2.2, JP1.10, JP1.2, JP1.4, JP1.6, JP1.8, RBAT38.1, RBAT39.1; no longer U$3.1_GND, U$3.GND2, U$5.1_GND, U$5.GND2
- net GYRO_1: now also AT328.28; no longer AT328.25
- net GYRO_2: now also AT328.27; no longer AT328.26
- net GYRO_3: now also AT328.26; no longer AT328.27
- net GYRO_4: now also AT328.25; no longer AT328.28
- net LEDG: now also LEDG.C, Q12.3; no longer Q12.1, RBAT29.2
- net LEDR: no longer LEDG.C, Q12.3, Q8.1, RBAT27.2
- net LED_G: now also Q12.1, RBAT29.2, U$4.36; no longer U$4.15, U$4.18
- net LED_R: now also Q8.1, RBAT27.2, U$4.32; no longer U$4.13, U$4.16
- net MISO_5V: no longer U$3.MISO, U$5.MISO
- net MOSI: now also IC2.17; no longer IC2.2
- net MOSI_5V: now also IC2.3; no longer IC2.18, U$3.MOSI, U$5.MOSI
- net N$15: now also PLUG_3.81_2.3; no longer PLUG_3.81_2.1
- net N$4: now also K1.S, PLUG_3.81_2.1; no longer U2.10
- net RAW_FUSED: no longer U$3.RAW, U$3.RAW2, U$5.RAW, U$5.RAW2
- net RAW_UNPROTECTED: now also JP1.1, JP1.3, JP1.5, JP1.7, JP1.9
- net REG_RCK: now also IC2.2; no longer U2.12
- net RELAY1: now also U$4.37; no longer U$4.12
- net RST1: now also RBAT9.1, U2.3; no longer RBAT4.1, U2.15
- net RST3: now also RBAT4.1, U2.15; no longer RBAT8.1, U2.2
- net RST4: now also RBAT8.1, U2.2; no longer RBAT9.1, U2.3
- net RST5: now also RBAT12.1, U2.6; no longer RBAT10.1, U2.4
- net RST6: now also RBAT13.1, U2.7; no longer RBAT11.1, U2.5
- net RST7: now also RBAT10.1, U2.4; no longer RBAT12.1, U2.6
- net RST8: now also RBAT11.1, U2.5; no longer RBAT13.1, U2.7
- net SCK: now also IC2.15; no longer IC2.11
- net SCK_5V: now also IC2.5, RBAT39.2; no longer IC2.9, U$3.SCK, U$5.SCK
- net TELECO_CS: now also IC2.11; no longer IC2.17
- net TELECO_CS_5V: now also IC2.9; no longer IC2.3
Routing:
- net +5V: track 32.4 -> 476.1 mm, vias 0 -> 5
- net SCK_5V: track 0.00 -> 208.9 mm, vias 0 -> 1
- net MOSI_5V: track 0.00 -> 207.4 mm, vias 0 -> 3
- net MISO_5V: track 0.00 -> 181.5 mm, vias 0 -> 4
- net PWM_LED_1: track 0.00 -> 137.2 mm, vias 0 -> 3
- net RAW_FUSED: track 114.6 -> 237.9 mm, vias 0 -> 1
- net EXT1_CS_5V: track 0.00 -> 115.7 mm, vias 0 -> 2
- net TELECO_CS_5V: track 0.00 -> 106.4 mm, vias 0 -> 1
- net EXT2_CS_5V: track 0.00 -> 104.2 mm, vias 0 -> 4
- net CODE: track 0.00 -> 102.5 mm, vias 0 -> 1
- net LEDR: track 0.00 -> 99.9 mm, vias 0 -> 2
- net LEDG: track 0.00 -> 97.0 mm, vias 0 -> 2
- net RX-I: track 0.00 -> 93.0 mm, vias 0 -> 1
- net TX-O: track 0.00 -> 86.3 mm, vias 0 -> 1
- net INT_TELECO: track 0.00 -> 77.8 mm, vias 0 -> 1
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- added copper zone on layer 1, net GND
- added copper zone on layer 16, net GND
Other:
- board size 99 x 87 mm -> 99 x 90 mm
