File: pcb/dnc_v1/dnc.brd (EAGLE design)
At the start: 97.2 x 88 mm, 143 parts, among them IC1 LM2596S, IC2 74ACT244SC, Q1 IRF9321PBF, Q10 FDN337N, Q11 FDN337N, Q12 BSS138, Q13 BSS138, Q14 FDN337N, Q2 BSS670, Q3 BSS138, Q4 BSS670, Q5 BSS138, Q6 BSS316, Q7 BSS138, Q8 BSS138, Q9 BSS670, U1 MAX202CDWR, U2 74HCT595D, U3 TC7SU04F, U4 AL8805WS, U5 AL8805WS, U6 TC7SU04F, X1 USB

Commit message: add telco sauvegarde prig
Connections:
- net N$14 renamed BB
- net N$15 renamed RNC
- net N$20 renamed S2
- net N$22 renamed S1
- net N$23 renamed S3
- net N$29 renamed RR
- net N$4 renamed RNO
- net N$9 renamed GG
Changed lines of the file:
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@@
 <wire x1="93.46" y1="49.43" x2="93.56" y2="50.165" width="0.3048" layer="1"/>
 </signal>
-<signal name="N$22">
+<signal name="S1">
 <contactref element="R6" pad="1"/>
 <contactref element="R9" pad="1"/>
@@
 <wire x1="3.175" y1="46.609" x2="3.2004" y2="46.6344" width="0.3048" layer="16"/>
 </signal>
-<signal name="N$20">
+<signal name="S2">
 <contactref element="R7" pad="1"/>
 <contactref element="R10" pad="1"/>
@@
 <wire x1="11.557" y1="30.305" x2="10.375" y2="30.305" width="0.3048" layer="1"/>
 </signal>
-<signal name="N$23">
+<signal name="S3">
 <contactref element="R8" pad="1"/>
 <contactref element="R11" pad="1"/>
@@
 <wire x1="70.485" y1="53.34" x2="70.485" y2="50.8" width="0.3048" layer="16"/>
 </signal>
-<signal name="N$4" class="4">
+<signal name="RNO" class="4">
 <contactref element="RELAY1" pad="S"/>
 <contactref element="RELAY" pad="1"/>
@@
 <wire x1="74.295" y1="1.905" x2="74.295" y2="0.762" width="1.27" layer="16"/>
 </signal>
-<signal name="N$15" class="4">
+<signal name="RNC" class="4">
 <contactref element="RELAY1" pad="O"/>
 <contactref element="RELAY" pad="3"/>
@@
 <wire x1="72.263" y1="76.835" x2="74.93" y2="79.502" width="0.6096" layer="1"/>
 </signal>
-<signal name="N$9">
+<signal name="GG">
 <contactref element="F3" pad="2"/>
 <contactref element="RGB-LED" pad="6"/>
@@
 <wire x1="43.815" y1="78.486" x2="43.561" y2="78.74" width="0.8128" layer="16"/>
 </signal>
-<signal name="N$14">
+<signal name="BB">
 <contactref element="F4" pad="2"/>
 <contactref element="RGB-LED" pad="8"/>
@@
 </polygon>
 </signal>
-<signal name="N$29">
+<signal name="RR">
 <contactref element="F5" pad="2"/>
 <contactref element="RGB-LED" pad="4"/>
