File: pcb/dnc_v1/dnc.sch (EAGLE design)
At the start: 66 parts, among them Q5 TSM2306CX, Q7 TSM2306CX, Q8 TSM2306CX

Commit message: avance sur v1
Parts:
- removed 3.3/5: (no value), SparkFun:M02PTH3
- removed EXT5, EXT6: EXT-DNC, pierre_vv:EXT-DNC
- removed MOS_TEMP: 200mA/50V, SparkFun-DiscreteSemi:MOSFET-NCHANNELBSS138
- removed PTC: (no value), ptc-ntc:PTC679
- removed REG1, REG2: 74HC595D, 74xx-eu:74HC595D
- removed RTEMP0: 100k, SparkFun-Passives:RESISTOR0603-RES
- removed RTEMP2: (no value), SparkFun-Passives:RESISTOR0603-RES
- removed U$5: DC/DC_SEED, pierre_vv:DC/DC_SEED
- added C1: (no value), rcl:CPOL-USE
- added C3, C4: 0.1uF, rcl:C-EUC0603
- added C5, C6: 1uF, rcl:C-EUC0603
- added D1: 40v5A, diode:SCHOTTKY-DIODESMC
- added D2: 1.8v, SparkFun-DiscreteSemi:DIODE-ZENERSOD-123
- added D3: 33v, SparkFun-DiscreteSemi:DIODE-ZENERSOD-123
- added IC1: LM2596S, national-semiconductor:LM2596S
- added L1: 100nH, SparkFun:INDUCTORPWR
- added Q1: IRF9321PBF, pierre_vv:IRF9321PBF
- added RBAT3: 100K, SparkFun-Passives:RESISTOR0603-RES
- added U1: AP2202-ADJ, SparkFun-PowerIC:AP2202-ADJ
- added U2: 74HCT595D, IC:74HCT595D
- added U3, U4: 74LVC1G08SE-7, SparkFun-DigitalIC:7408SE
- C2: value 10uF -> 680uF30mm; device SparkFun:CAP_POL1206 -> SparkFun:CAP_POLPTH4
- F1: value PTCPTH -> 8A; device SparkFun-PowerIC:PTCPTH -> SparkFun:PTCPTH
- RBAT1: value 100k -> 100k1%
- RBAT2: value 10k -> 10k1%
Connections:
- removed net ACTIVE_ANALOG_TEMP: MOS_TEMP.G, RTEMP0.1
- removed net N$10: EXT5.FREE
- removed net N$11: MOS_TEMP.D, PTC.2
- removed net N$12: F1.1, RAW_IN.1
- removed net N$7: REG1A.QH*, REG2A.SER
- removed net N$9: EXT6.FREE
- removed net RAW: C2.+, EXT1.RAW, EXT2.RAW, EXT3.RAW, EXT4.RAW, EXT5.RAW, EXT6.RAW, F1.2, MOS_PWR1.D, MOS_PWR2.D, MOS_PWR3.D, RBAT1.2, U$5.IN+
- removed net RST10: REG2A.QB
- removed net RST11: REG2A.QC
- removed net RST12: REG2A.QD
- removed net RST13: REG2A.QE
- removed net RST14: REG2A.QF
- removed net RST15: REG2A.QG
- removed net RST16: REG2A.QH
- removed net RST9: REG2A.QA
- new net MOSI_5V: TITREUR1.7, TITREUR2.7, U4.Y
- new net N$1: D1.C, IC1.OUT, L1.1
- new net PROTECT_GATE: D2.A, Q1.G, RBAT3.1
- new net RAW_FUSED: C2.+, C3.1, EXT1.RAW, EXT2.RAW, EXT3.RAW, EXT4.RAW, F1.2, IC1.VIN, MOS_PWR1.D, MOS_PWR2.D, MOS_PWR3.D, RBAT1.2
- new net RAW_POL_PROTECTED: D2.C, D3.C, F1.1, Q1.S
- new net RAW_UNPROTECTED: Q1.D, RAW_IN.1
- new net SCK_TITREUR: TITREUR1.5, TITREUR2.5, U3.Y
- net +3V3: now also C6.1, U1.OUT; no longer 3.3/5.1, EXT5.3.3V, EXT6.3.3V
- net +5V: now also C1.+, C4.1, C5.1, IC1.FB, L1.2, U1.EN, U1.IN, U2.SCL, U2.VCC, U3.VCC, U4.A, U4.VCC; no longer 3.3/5.2, EXT5.5V, EXT6.5V, PTC.1, U$5.OUT+
- net /CS_EXT_5: no longer EXT5.RST
- net /CS_EXT_6: no longer EXT6.RST
- net ANALOG_TEMP: no longer MOS_TEMP.S, RTEMP2.1
- net CODE: no longer EXT5.COD, EXT6.COD
- net GND: now also C1.-, C3.2, C4.2, C5.2, C6.2, D1.A, D3.A, IC1.!ON!/OFF, IC1.GND, RBAT3.2, U1.GND, U2.G, U2.GND, U3.GND, U4.GND; no longer EXT5.GND, EXT6.GND, REG1A.G, REG2A.G, RTEMP0.2, RTEMP2.2, U$5.IN-, U$5.OUT-
- net MISO: no longer EXT5.MISO, EXT6.MISO
- net MOSI: now also U4.B; no longer EXT5.MOSI, EXT6.MOSI, REG1A.SER, TITREUR1.7, TITREUR2.7
- net REG_CLR: no longer REG1A.SCL, REG2A.SCL
- net REG_RCK: now also U3.A; no longer REG1A.RCK, REG2A.RCK
- net RST1: now also U2.QA; no longer REG1A.QA
- net RST2: now also U2.QB; no longer REG1A.QB
- net RST3: now also U2.QC; no longer REG1A.QC
- net RST4: now also U2.QD; no longer REG1A.QD
- net RST5: now also U2.QE; no longer REG1A.QE
- net RST6: now also U2.QF; no longer REG1A.QF
- net RST7: now also U2.QG; no longer REG1A.QG
- net RST8: now also U2.QH; no longer REG1A.QH
- net SCK: now also U2.SCK, U3.B; no longer EXT5.SCK, EXT6.SCK, REG1A.SCK, REG2A.SCK, TITREUR1.5, TITREUR2.5
Other:
- note added: "5V buck converter and 3.3V LDO"
- note added: "CS titreur driver"
- note added: "reverse + overvoltage protection"
- moved on the sheet: 8MHZ, AT328, C2, C3.3, CMHZ, CRST, F1, ISP, MOS_BAT, PROG1, RAW_IN, RBAT0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

Commit message: in progress
Parts:
- removed 8MHZ: RESONATOR, pierre_vv:RESONATOR
- removed A_IN1, A_IN2, A_IN3: DNC_IN3, pierre_vv:DNC_IN3
- removed IN1, IN2, IN3, IN4, OUT1, OUT2, OUT3: DNC_IN2, pierre_vv:DNC_IN2
- removed MOS_PWR1, MOS_PWR2, MOS_PWR3, Q5, Q7, Q8: TSM2306CX, SparkFun-DiscreteSemi:MOSFET-NCHANNEL2N7002PW
- removed PWR_OUT1, PWR_OUT2, PWR_OUT3: DNC_IN2PWR, pierre_vv:DNC_IN2PWR
- removed RIN1, RIN2, RIN3, RIN4: (no value), SparkFun-Passives:RESISTOR0603-RES
- removed RIN10, RIN8, RIN9, ROUT1, ROUT2, ROUT3: 100k, SparkFun-Passives:RESISTOR0603-RES
- added 16MHZ: 16MHZ, SparkFun-FreqCtrl:RESONATOR16MHZ
- added C10, C8: 1uF, rcl:C-EUC0603
- added C7, C9: 0.1uF, rcl:C-EUC0603
- added D4, D5: 40v5A, diode:SCHOTTKY-DIODESMC
- added IC2: 74S244DW, 74xx-us:74S244DW
- added L2, L3: 100nH, SparkFun:INDUCTORPWR
- added PLUG_3.81_1: FLEX, pierre_vv:M03
- added PLUG_3.81_2_1: LED10W2, pierre_vv:M02PLUG
- added PLUG_3.81_2_2: LED10W1, pierre_vv:M02PLUG
- added PLUG_3.81_6_1: M06, pierre_vv:M06
- added Q10, Q11, Q2, Q4, Q6, Q9: BSS670, SparkFun-DiscreteSemi:MOSFET-NCHANNELBSS138
- added Q3: BSS138, SparkFun-DiscreteSemi:MOSFET-NCHANNELBSS138
- added RBAT10, RBAT11, RBAT12, RBAT13, RBAT16, RBAT17, RBAT18, RBAT19, RBAT20, RBAT21, RBAT4, RBAT5, RBAT8, RBAT9: 100K, SparkFun-Passives:RESISTOR0603-RES
- added RBAT14, RBAT15: 0.110, SparkFun-Passives:RESISTOR0603-RES
- added RBAT22, RBAT23, RBAT24, RBAT25, RBAT6, RBAT7: 10K, SparkFun-Passives:RESISTOR0603-RES
- added SJ1, SJ2: JUMPER-PTH-2-NC, SparkFun-Passives:JUMPER-PTH-2-NC
- added U5: AL8807, SparkFun-PowerIC:AL8805
- AT328: value ATMEGA168 -> ATMEGA328
- MOS_BAT: value 200mA/50V -> MOSFET-NCHANNELBSS138
- U3: value 74LVC1G08SE-7 -> TC7SU04F; device SparkFun-DigitalIC:7408SE -> SparkFun-DigitalIC:INVERTER_SOT23-5
- U4: value 74LVC1G08SE-7 -> AL8807; device SparkFun-DigitalIC:7408SE -> SparkFun-PowerIC:AL8805
Connections:
- net REG_CLR renamed LED_R
- removed net /CS_EXT_5: U$4.GPIO2
- removed net /CS_EXT_6: U$4.GND_4
- removed net ACTIVE_OUT_1: Q5.G, RIN8.2, U$4.GPIO16
- removed net ACTIVE_OUT_2: Q7.G, RIN9.2, U$4.GPIO20
- removed net ACTIVE_OUT_3: Q8.G, RIN10.2, U$4.GPIO21
- removed net ACTIVE_OUT_POWER_1: AT328.PD2(INT0), MOS_PWR1.G, ROUT1.2
- removed net ACTIVE_OUT_POWER_2: AT328.PD3(INT1), MOS_PWR2.G, ROUT2.2
- removed net ACTIVE_OUT_POWER_3: AT328.PD6(AIN0), MOS_PWR3.G, ROUT3.2
- removed net ANALOG_IN_1: AT328.PC3(ADC3), A_IN1.3
- removed net ANALOG_IN_2: AT328.PC4(ADC4/SDA), A_IN2.3
- removed net ANALOG_IN_3: AT328.PC5(ADC5/SCL), A_IN3.3
- removed net ANALOG_TEMP: AT328.PC2(ADC2)
- removed net IN_1: IN1.2, RIN1.2, U$4.GPIO26
- removed net IN_2: IN2.2, RIN2.2, U$4.GPIO19
- removed net IN_3: IN3.2, RIN3.2, U$4.GPIO13
- removed net IN_4: IN4.2, RIN4.2, U$4.GPIO6
- removed net OUT_1: OUT1.1, Q5.S
- removed net OUT_2: OUT2.1, Q7.S
- removed net OUT_3: OUT3.1, Q8.S
- removed net OUT_POWER_1: MOS_PWR1.S, PWR_OUT1.1
- removed net OUT_POWER_2: MOS_PWR2.S, PWR_OUT2.1
- removed net OUT_POWER_3: MOS_PWR3.S, PWR_OUT3.1
- removed net SCK_TITREUR: TITREUR1.5, TITREUR2.5, U3.Y
- new net ALL_CS_ENABLE_ACTIVE_LOW: IC2A.G, IC2B.G, U2.G, U3.Y
- new net ATMEGA_CS_5V: AT328.PB2(SS/OC1B), IC2B.Y3
- new net CS_TRIGGER_ACTIVE_HIGH: U$4.GPIO26, U3.A
- new net EXT1_CS: IC2A.A1, U$4.GPIO2
- new net EXT1_CS_5V: IC2A.Y1
- new net EXT2_CS: IC2A.A2, U$4.GPIO3
- new net EXT2_CS_5V: IC2A.Y2
- new net EXT3_CS: IC2A.A3, U$4.GPIO4
- new net EXT3_CS_5V: IC2A.Y3
- new net EXT4_CS: IC2B.A2, IC2B.Y2, U$4.GPIO5
- new net EXT5_CS: U$4.GPIO6
- new net GYRO_1: AT328.PC2(ADC2), Q4.G, RBAT16.2
- new net GYRO_2: AT328.PC3(ADC3), Q2.G, RBAT17.2
- new net GYRO_3: AT328.PC4(ADC4/SDA), Q6.G, RBAT18.2
- new net GYRO_4: AT328.PC5(ADC5/SCL), Q9.G, RBAT19.2
- new net INT_ATMEGA: RBAT22.1, RBAT23.2, U$4.GPIO20
- new net INT_ATMEGA_5V: AT328.PD4(XCK/T0), RBAT22.2
- new net INT_TELECO: RBAT24.1, RBAT25.2, U$4.GPIO21
- new net INT_TELECO_5V: RBAT24.2
- new net LED+1: C8.1, PLUG_3.81_2_1.1, RBAT14.1, SJ1.2, U4.SET
- new net LED+2: C10.1, PLUG_3.81_2_2.1, RBAT15.1, SJ2.2, U5.SET
- new net LED-1: C8.2, L2.2, PLUG_3.81_2_1.2
- new net LED-2: C10.2, L3.2, PLUG_3.81_2_2.2
- new net LED_G: U$4.GPIO22
- new net MISO_5V: AT328.PB4(MISO), ISP.1, Q3.D, RBAT7.1
- new net N$10: PLUG_3.81_6_1.2, Q4.D
- new net N$11: PLUG_3.81_6_1.3, Q2.D
- new net N$12: PLUG_3.81_6_1.4, Q6.D
- new net N$13: PLUG_3.81_6_1.5, Q9.D
- new net N$14: PLUG_3.81_1.2, Q10.D
- new net N$15: EXT1.5V, EXT2.5V, EXT3.5V, EXT4.5V
- new net N$16: AT328.PD2(INT0)
- new net N$6: D4.A, L2.1, U4.SW
- new net N$7: D5.A, L3.1, U5.SW
- new net N$9: PLUG_3.81_1.3, Q11.D
- new net PWM_FLEX_1: AT328.PD3(INT1), Q10.G, RBAT20.2
- new net PWM_FLEX_2: AT328.PB1(OC1A), Q11.G, RBAT21.2
- new net PWM_LED_1: AT328.PD5(T1), U5.CTRL
- new net PWM_LED_2: AT328.PD6(AIN0), U4.CTRL
- new net RESET_5V: AT328.PC6(/RESET), ISP.5
- new net SCK_5V: AT328.PB5(SCK), IC2B.Y1, ISP.3, TITREUR1.5, TITREUR2.5
- new net TELECO_CS: IC2B.A4, U$4.GPIO19
- new net TELECO_CS_5V: IC2B.Y4
- net +3V3: now also Q3.G, RBAT6.2; no longer AT328.AVCC, AT328.VCC@1, AT328.VCC@2, A_IN1.2, A_IN2.2, A_IN3.2, C3.3.1, IN1.1, IN2.1, IN3.1, IN4.1, ISP.2, PROG1.VCC, RRST.2
- net +5V: now also AT328.AVCC, AT328.VCC@1, AT328.VCC@2, C3.3.1, IC2P.VCC, ISP.2, PROG1.VCC, RBAT10.2, RBAT11.2, RBAT12.2, RBAT13.2, RBAT4.2, RBAT5.2, RBAT7.2, RBAT8.2, RBAT9.2, RRST.2; no longer EXT1.5V, EXT2.5V, EXT3.5V, EXT4.5V, Q5.D, Q7.D, Q8.D, U4.A, U4.VCC
- net /CS_EXT_1: no longer U$4.GPIO12
- net /CS_EXT_2: no longer U$4.GPIO5
- net /CS_EXT_3: no longer U$4.GPIO4
- net /CS_EXT_4: no longer U$4.GPIO3
- net ACTIVE_ANALOG_RAW: no longer AT328.PD4(XCK/T0)
- net ATMEGA_CS: now also IC2B.A3, U$4.GPIO13; no longer AT328.PB2(SS/OC1B), U$4.GPIO23
- net GND: now also 16MHZ.2, C7.2, C9.2, IC2P.GND, Q10.S, Q11.S, Q2.S, Q4.S, Q6.S, Q9.S, RBAT16.1, RBAT17.1, RBAT18.1, RBAT19.1, RBAT20.1, RBAT21.1, RBAT23.1, RBAT25.1, U$4.GND_4, U5.GND; no longer 8MHZ.2, A_IN1.1, A_IN2.1, A_IN3.1, OUT1.2, OUT2.2, OUT3.2, PWR_OUT1.2, PWR_OUT2.2, PWR_OUT3.2, RIN1.1, RIN10.1, RIN2.1, RIN3.1, RIN4.1, RIN8.1, RIN9.1, ROUT1.1, ROUT2.1, ROUT3.1, U2.G
- net MISO: now also Q3.S, RBAT6.1; no longer AT328.PB4(MISO), ISP.1
- net MOSI: now also IC2A.A4; no longer AT328.PB3(MOSI/OC2), ISP.4, U4.B
- net MOSI_5V: now also AT328.PB3(MOSI/OC2), IC2A.Y4, ISP.4; no longer U4.Y
- net N$43: now also 16MHZ.1; no longer 8MHZ.1
- net N$44: now also 16MHZ.3; no longer 8MHZ.3
- net RAW_FUSED: now also C7.1, C9.1, D4.C, D5.C, PLUG_3.81_1.1, PLUG_3.81_6_1.1, PLUG_3.81_6_1.6, RBAT14.2, RBAT15.2, SJ1.1, SJ2.1, U4.VIN, U5.VIN; no longer MOS_PWR1.D, MOS_PWR2.D, MOS_PWR3.D
- net REG_RCK: no longer U3.A
- net RESET: no longer AT328.PC6(/RESET), ISP.5
- net RST1: now also RBAT4.1
- net RST2: now also RBAT5.1
- net RST3: now also RBAT8.1
- net RST4: now also RBAT9.1
- net RST5: now also RBAT10.1
- net RST6: now also RBAT11.1
- net RST7: now also RBAT12.1
- net RST8: now also RBAT13.1
- net SCK: now also IC2B.A1; no longer AT328.PB5(SCK), ISP.3, U3.B
Other:
- note added: "1x FLEX DRIVER"
- note added: "2X LED 10W DRIVER"
- note added: "4x FLEX GYRO on/off DRIVER"
- note added: "LEVEL SHIFT 3.3V TO 5V"
- note added: "RPI DOCK"
- moved on the sheet: A+_UART, C3.3, U4

Commit message: in progress 2
Parts:
- removed EXT1, EXT2, EXT3, EXT4: EXT-DNC, pierre_vv:EXT-DNC
- added U$1: EXT1, pierre_vv:EXT-DNC
- added U$2: EXT2, pierre_vv:EXT-DNC
- added U$3: EXT3, pierre_vv:EXT-DNC
- added U$5: EXT4, pierre_vv:EXT-DNC
- added U$8: RJ45-EXTDNC, con-amphenol-rj45-ld:RJ45-EXTDNC
- C3.3, CMHZ, CRST: device rcl:C-EUC0805 -> rcl:C-EUC0603
- RBAT23, RBAT25: value 10K -> 20K
Connections:
- removed net /CS_EXT_1: EXT1.RST
- removed net /CS_EXT_2: EXT2.RST
- removed net /CS_EXT_3: EXT3.RST
- removed net /CS_EXT_4: EXT4.RST
- removed net N$15: EXT1.5V, EXT2.5V, EXT3.5V, EXT4.5V
- removed net N$21: EXT1.FREE
- removed net N$4: EXT2.FREE
- removed net N$5: EXT3.FREE
- removed net N$8: EXT4.FREE
- new net EXT4_CS_5V: U$5.CS
- net +3V3: no longer EXT1.3.3V, EXT2.3.3V, EXT3.3.3V, EXT4.3.3V
- net +5V: now also U$1.5V, U$2.5V, U$3.5V, U$5.5V, U$8.5V
- net CODE: now also U$1.COD, U$2.COD, U$3.COD, U$5.COD, U$8.COD; no longer EXT1.COD, EXT2.COD, EXT3.COD, EXT4.COD
- net EXT1_CS_5V: now also U$1.CS
- net EXT2_CS_5V: now also U$2.CS
- net EXT3_CS_5V: now also U$3.CS
- net GND: now also U$1.GND, U$2.GND, U$3.GND, U$5.GND, U$8.GND; no longer EXT1.GND, EXT2.GND, EXT3.GND, EXT4.GND
- net INT_TELECO_5V: now also U$8.INT
- net MISO: no longer EXT1.MISO, EXT2.MISO, EXT3.MISO, EXT4.MISO
- net MISO_5V: now also U$1.MISO, U$2.MISO, U$3.MISO, U$5.MISO, U$8.MISO
- net MOSI: no longer EXT1.MOSI, EXT2.MOSI, EXT3.MOSI, EXT4.MOSI
- net MOSI_5V: now also U$1.MOSI, U$2.MOSI, U$3.MOSI, U$5.MOSI, U$8.MOSI
- net RAW_FUSED: now also U$1.RAW, U$2.RAW, U$3.RAW, U$5.RAW; no longer EXT1.RAW, EXT2.RAW, EXT3.RAW, EXT4.RAW
- net SCK: no longer EXT1.SCK, EXT2.SCK, EXT3.SCK, EXT4.SCK, U2.SCK
- net SCK_5V: now also U$1.SCK, U$2.SCK, U$3.SCK, U$5.SCK, U$8.SCK, U2.SCK
- net TELECO_CS_5V: now also U$8./CS
Other:
- note added: "2x FLEX DRIVER"
- note removed: "1x FLEX DRIVER"
- moved on the sheet: 16MHZ, AT328, C10, C3.3, C7, C8, C9, CMHZ, CRST, D4, D5, ISP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

Commit message: schematic fini début routage
Parts:
- removed C5, C6: 1uF, rcl:C-EUC0603
- removed MOS_BAT: MOSFET-NCHANNELBSS138, SparkFun-DiscreteSemi:MOSFET-NCHANNELBSS138
- removed U1: AP2202-ADJ, SparkFun-PowerIC:AP2202-ADJ
- added C11, C12, C13: 1uF, rcl:C-EUC0603
- added C3.1: 0.1uF, rcl:C-EUC0603
- added D6: (no value), SparkFun-DiscreteSemi:DIODESMA-ALT
- added K1: G5L, relay:G5L
- added LEDG, LEDR: (no value), led:LEDCHIPLED_0603
- added PLUG_3.81_2: FLEX, pierre_vv:M03
- added Q12, Q5, Q7, Q8: BSS138, SparkFun-DiscreteSemi:MOSFET-NCHANNELBSS138
- added RBAT26, RBAT27, RBAT29: 100K, SparkFun-Passives:RESISTOR0603-RES
- added RBAT28, RBAT30: 220, SparkFun-Passives:RESISTOR0603-RES
- added RBAT31, RBAT32, RBAT35: 56K, SparkFun-Passives:RESISTOR0603-RES
- added RBAT33, RBAT34, RBAT36: 33K, SparkFun-Passives:RESISTOR0603-RES
- added RBAT37: 1K, SparkFun-Passives:RESISTOR0603-RES
- added S1: (no value), switch-omron:31-XX
- added U$6: M08, pierre_vv:M08
- Q10, Q11: value BSS670 -> BSS316
Connections:
- removed net N$16: AT328.PD2(INT0)
- removed net RESET_5V: AT328.PC6(/RESET), ISP.5
- new net FLOAT1: AT328.ADC6, U$6.2
- new net FLOAT2: AT328.ADC7, U$6.3
- new net LEDG: Q12.G, RBAT29.2
- new net LEDR: LEDG.C, LEDR.C, Q12.D, Q8.D, Q8.G, RBAT27.2
- new net N$15: K12.O, PLUG_3.81_2.1
- new net N$17: K12.S, PLUG_3.81_2.3
- new net N$18: LEDG.A, RBAT30.1
- new net N$19: U$4.GPIO25
- new net N$20: RBAT32.1, RBAT34.1, U$6.6
- new net N$21: LEDR.A, RBAT28.1
- new net N$22: RBAT31.1, RBAT33.1, S1.S, U$6.7
- new net N$23: RBAT35.1, RBAT36.1, U$6.5
- new net N$25: RBAT37.1, U$6.1
- new net N$4: U2.SCL
- new net N$5: D6.A, K11.2, Q5.D
- new net N$8: K12.P, PLUG_3.81_2.2
- new net PUSH1: AT328.PD2(INT0), C13.1, RBAT33.2
- new net PUSH2: AT328.PD7(AIN1), C12.1, RBAT34.2
- new net PUSH3: AT328.PB0(ICP), C11.1, RBAT36.2
- new net RELAY1: Q5.G, RBAT26.2, U$4.GPIO18
- net +3V3: no longer C6.1, U$4.GPIO24, U1.OUT
- net +5V: now also C3.1.1, D6.C, K11.1, RBAT28.2, RBAT30.2, RBAT31.2, RBAT32.2, RBAT35.2, RBAT37.2; no longer C5.1, U1.EN, U1.IN, U2.SCL
- net ACTIVE_ANALOG_RAW: now also Q7.G; no longer MOS_BAT.G
- net ANALOG_RAW: now also Q7.S; no longer MOS_BAT.S
- net EXT1_CS: now also IC2A.A4; no longer IC2A.A1
- net EXT1_CS_5V: now also IC2A.Y4; no longer IC2A.Y1
- net EXT2_CS: now also IC2A.A3; no longer IC2A.A2
- net EXT2_CS_5V: now also IC2A.Y3; no longer IC2A.Y2
- net EXT3_CS: now also IC2A.A2; no longer IC2A.A3
- net EXT3_CS_5V: now also IC2A.Y2; no longer IC2A.Y3
- net GND: now also C11.2, C12.2, C13.2, C3.1.2, Q12.S, Q5.S, Q8.S, RBAT26.1, RBAT27.1, RBAT29.1, S1.P, U$6.4, U$6.8; no longer C5.2, C6.2, U1.GND
- net LED_G: now also U$4.GPIO24
- net LED_R: now also U$4.GPIO23
- net MOSI: now also IC2A.A1; no longer IC2A.A4
- net MOSI_5V: now also IC2A.Y1, U2.SER; no longer IC2A.Y4
- net N$3: now also Q7.D; no longer MOS_BAT.D
- net REG_RCK: now also U2.RCK
- net RESET: now also AT328.PC6(/RESET), ISP.5
Other:
- note added: "LEDS"
- note added: "RELAY"
- moved on the sheet: 16MHZ, A+_UART, AT328, C1, C10, C2, C3, C3.3, C4, C7, C8, C9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

Commit message: routage terminé
Parts:
- removed U$3: EXT3, pierre_vv:EXT-DNC
- removed U$5: EXT4, pierre_vv:EXT-DNC
- added C3.2: 0.1uF, rcl:C-EUC0603
- added JP1: M05X2SHD_LOCK, SparkFun:M05X2SHD_LOCK
- added RBAT38, RBAT39: 10K, SparkFun-Passives:RESISTOR0603-RES
- PLUG_3.81_2: value FLEX -> RELAY
- SJ1, SJ2: value JUMPER-PTH-2-NC -> JUMPER-PTH-2-NO; device SparkFun-Passives:JUMPER-PTH-2-NC -> SparkFun-Passives:JUMPER-PTH-2-NO
Connections:
- net ALL_CS_ENABLE_ACTIVE_LOW renamed ALL_CS_ENABLE_ACTIVE_LOW_5V
- removed net ACTIVE_ANALOG_RAW: Q7.G, RBAT0.2
- removed net EXT4_CS: IC2B.A2, IC2B.Y2, U$4.GPIO5
- removed net EXT4_CS_5V: U$5.CS
- removed net EXT5_CS: U$4.GPIO6
- removed net N$17: K12.S, PLUG_3.81_2.3
- removed net N$19: U$4.GPIO25
- removed net N$5: D6.A, K11.2, Q5.D
- new net N$16: D6.A, K11.1, Q5.D
- new net READ_BATTERY: Q7.G, RBAT0.2, U$4.GPIO25
- new net REG_RCK_5V: IC2A.Y1, U2.RCK
- net +5V: now also C3.2.1, K11.2, U2.SCL; no longer K11.1, U$3.5V, U$5.5V
- net ATMEGA_CS: now also IC2B.A2; no longer IC2B.A3
- net ATMEGA_CS_5V: now also IC2B.Y2; no longer IC2B.Y3
- net CODE: no longer U$3.COD, U$5.COD
- net CS_TRIGGER_ACTIVE_HIGH: now also RBAT38.2, U$4.GPIO5; no longer U$4.GPIO26
- net EXT3_CS_5V: no longer U$3.CS
- net GND: now also C3.2.2, JP1.10, JP1.2, JP1.4, JP1.6, JP1.8, RBAT38.1, RBAT39.1; no longer U$3.GND, U$5.GND
- net GYRO_1: now also AT328.PC5(ADC5/SCL); no longer AT328.PC2(ADC2)
- net GYRO_2: now also AT328.PC4(ADC4/SDA); no longer AT328.PC3(ADC3)
- net GYRO_3: now also AT328.PC3(ADC3); no longer AT328.PC4(ADC4/SDA)
- net GYRO_4: now also AT328.PC2(ADC2); no longer AT328.PC5(ADC5/SCL)
- net LEDG: now also LEDG.C, Q12.D; no longer Q12.G, RBAT29.2
- net LEDR: no longer LEDG.C, Q12.D, Q8.G, RBAT27.2
- net LED_G: now also Q12.G, RBAT29.2, U$4.GPIO16; no longer U$4.GPIO22, U$4.GPIO24
- net LED_R: now also Q8.G, RBAT27.2, U$4.GPIO12; no longer U$4.GPIO23, U$4.GPIO27
- net MISO_5V: no longer U$3.MISO, U$5.MISO
- net MOSI: now also IC2B.A4; no longer IC2A.A1
- net MOSI_5V: now also IC2B.Y4; no longer IC2A.Y1, U$3.MOSI, U$5.MOSI
- net N$15: now also PLUG_3.81_2.3; no longer PLUG_3.81_2.1
- net N$4: now also K12.S, PLUG_3.81_2.1; no longer U2.SCL
- net RAW_FUSED: no longer U$3.RAW, U$5.RAW
- net RAW_UNPROTECTED: now also JP1.1, JP1.3, JP1.5, JP1.7, JP1.9
- net REG_RCK: now also IC2A.A1; no longer U2.RCK
- net RELAY1: now also U$4.GPIO26; no longer U$4.GPIO18
- net RST1: now also RBAT9.1, U2.QD; no longer RBAT4.1, U2.QA
- net RST3: now also RBAT4.1, U2.QA; no longer RBAT8.1, U2.QC
- net RST4: now also RBAT8.1, U2.QC; no longer RBAT9.1, U2.QD
- net RST5: now also RBAT12.1, U2.QG; no longer RBAT10.1, U2.QE
- net RST6: now also RBAT13.1, U2.QH; no longer RBAT11.1, U2.QF
- net RST7: now also RBAT10.1, U2.QE; no longer RBAT12.1, U2.QG
- net RST8: now also RBAT11.1, U2.QF; no longer RBAT13.1, U2.QH
- net SCK: now also IC2B.A3; no longer IC2B.A1
- net SCK_5V: now also IC2B.Y3, RBAT39.2; no longer IC2B.Y1, U$3.SCK, U$5.SCK
- net TELECO_CS: now also IC2B.A1; no longer IC2B.A4
- net TELECO_CS_5V: now also IC2B.Y1; no longer IC2B.Y4
Other:
- moved on the sheet: K1, RCODE

Commit message: maj + ajout rs232
Parts:
- removed C3.3, CMHZ: 0.1uF, rcl:C-EUC0603
- removed RBAT0, RBAT3: 100K, SparkFun-Passives:RESISTOR0603-RES
- removed RBAT1: 100k1%, SparkFun-Passives:RESISTOR0603-RES
- removed RBAT2: 10k1%, SparkFun-Passives:RESISTOR0603-RES
- removed RBAT31, RBAT32, RBAT35: 56K, SparkFun-Passives:RESISTOR0603-RES
- removed RBAT33, RBAT34, RBAT36: 33K, SparkFun-Passives:RESISTOR0603-RES
- removed RBAT37: 1K, SparkFun-Passives:RESISTOR0603-RES
- added C14, C15, C16, C17, C18, C5, C6: 0.1uF, rcl:C-EUC0603
- added JP2: regrck, SparkFun-Connectors:M01PTH
- added JP3: atmega cs, SparkFun-Connectors:M01PTH
- added JP4: allcs, SparkFun-Connectors:M01PTH
- added R0, R3: 100K, SparkFun-Passives:RESISTOR0603-RES
- added R1: 100k1%, SparkFun-Passives:RESISTOR0603-RES
- added R2: 10k1%, SparkFun-Passives:RESISTOR0603-RES
- added R31, R32, R35: 56K, SparkFun-Passives:RESISTOR0603-RES
- added R33, R34, R36: 33K, SparkFun-Passives:RESISTOR0603-RES
- added R37: 1K, SparkFun-Passives:RESISTOR0603-RES
- added RS232: (no value), SparkFun-Connectors:M03LOCK_LONGPADS
- added U1: MAX202CDWR, SparkFun-DigitalIC:MAX232SOIC16
- JP1: value M05X2SHD_LOCK -> CHARGEUR
- PLUG_3.81_6_1: value M06 -> GYRO LED
- renumbered K1 to RELAY1, RBAT10 to R10, RBAT11 to R11, RBAT12 to R12, RBAT13 to R13, RBAT14 to R14, RBAT15 to R15, RBAT16 to R16, RBAT17 to R17, RBAT18 to R18, RBAT19 to R19, RBAT20 to R20, RBAT21 to R21, RBAT22 to R22, RBAT23 to R23, RBAT24 to R24, RBAT25 to R25, RBAT27 to R27, RBAT28 to R28, RBAT29 to R29, RBAT30 to R30, RBAT38 to R38, RBAT39 to R39, RBAT4 to R4, RBAT5 to R5, RBAT6 to R6, RBAT7 to R7, RBAT8 to R8, RBAT9 to R9, U$1 to EXT1, U$2 to EXT2
Connections:
- new net N$24: C14.2, U1.V+
- new net N$35: C17.1, U1.V-
- new net N$50: C6.2, U1.C2-
- new net N$51: C6.1, U1.C2+
- new net N$52: C5.2, U1.C1-
- new net N$53: C5.1, U1.C1+
- new net PRXD_PIN2_RS232: RS232.1, U1.T2OUT
- new net PTXD_PIN3_RS232: RS232.2, U1.R2IN
- net +5V: now also C14.1, C15.1, C18.1, R31.2, R32.2, R35.2, R37.2, U1.VCC; no longer C3.3.1, RBAT31.2, RBAT32.2, RBAT35.2, RBAT37.2
- net ALL_CS_ENABLE_ACTIVE_LOW_5V: now also JP4.1
- net ANALOG_RAW: now also R2.2; no longer RBAT2.2
- net AREF: now also C16.1; no longer CMHZ.1
- net ATMEGA_CS_5V: now also JP3.1
- net GND: now also C15.2, C16.2, C17.2, C18.2, R0.1, R2.1, R3.2, RS232.3, U1.GND; no longer C3.3.2, CMHZ.2, RBAT0.1, RBAT2.1, RBAT3.2
- net N$20: now also R32.1, R34.1; no longer RBAT32.1, RBAT34.1
- net N$22: now also R31.1, R33.1; no longer RBAT31.1, RBAT33.1
- net N$23: now also R35.1, R36.1; no longer RBAT35.1, RBAT36.1
- net N$25: now also R37.1; no longer RBAT37.1
- net N$3: now also R1.1; no longer RBAT1.1
- net PROTECT_GATE: now also R3.1; no longer RBAT3.1
- net PUSH1: now also R33.2; no longer RBAT33.2
- net PUSH2: now also R34.2; no longer RBAT34.2
- net PUSH3: now also R36.2; no longer RBAT36.2
- net RAW_FUSED: now also R1.2; no longer RBAT1.2
- net READ_BATTERY: now also R0.2; no longer RBAT0.2
- net REG_RCK_5V: now also JP2.1
- net RXA+: now also U1.R2OUT
- net TXA+: now also U1.T2IN
Other:
- note added: "INPUT 3D and 2A"
- note added: "RS232"
- moved on the sheet: 16MHZ, AT328, C1, C11, C12, C13, C2, C3, C4, D1, D2, D3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
