File: pcb/dnc_v1/dnc.sch (EAGLE design)
At the start: 143 parts, among them IC1 LM2596S, IC2 74ACT244SC, Q1 IRF9321PBF, Q10 FDN337N, Q11 FDN337N, Q12 BSS138, Q13 BSS138, Q14 FDN337N, Q2 BSS670, Q3 BSS138, Q4 BSS670, Q5 BSS138, Q6 BSS316, Q7 BSS138, Q8 BSS138, Q9 BSS670, U1 MAX202CDWR, U2 74HCT595D, U3 TC7SU04F, U4 AL8805WS, U5 AL8805WS, U6 TC7SU04F, X1 USB

Commit message: add telco sauvegarde prig
Connections:
- net N$14 renamed BB
- net N$15 renamed RNC
- net N$20 renamed S2
- net N$22 renamed S1
- net N$23 renamed S3
- net N$29 renamed RR
- net N$4 renamed RNO
- net N$9 renamed GG
Changed lines of the file:
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@@
 </segment>
 </net>
-<net name="N$22" class="0">
+<net name="S1" class="0">
 <segment>
 <pinref part="R6" gate="G$1" pin="1"/>
@@
 </segment>
 </net>
-<net name="N$20" class="0">
+<net name="S2" class="0">
 <segment>
 <pinref part="R7" gate="G$1" pin="1"/>
@@
 </segment>
 </net>
-<net name="N$23" class="0">
+<net name="S3" class="0">
 <segment>
 <pinref part="R8" gate="G$1" pin="1"/>
@@
 </segment>
 </net>
-<net name="N$4" class="4">
+<net name="RNO" class="4">
 <segment>
 <pinref part="RELAY1" gate="2" pin="S"/>
@@
 </segment>
 </net>
-<net name="N$15" class="4">
+<net name="RNC" class="4">
 <segment>
 <pinref part="RELAY1" gate="2" pin="O"/>
@@
 </segment>
 </net>
-<net name="N$9" class="0">
+<net name="GG" class="0">
 <segment>
 <pinref part="F3" gate="G$1" pin="2"/>
@@
 </segment>
 </net>
-<net name="N$14" class="0">
+<net name="BB" class="0">
 <segment>
 <pinref part="F4" gate="G$1" pin="2"/>
@@
 </segment>
 </net>
-<net name="N$29" class="0">
+<net name="RR" class="0">
 <segment>
 <pinref part="F5" gate="G$1" pin="2"/>
