File: pcb/pieuvre/dnc.sch (EAGLE design)
At the start: 143 parts, among them IC1 LM2596S, IC2 74ACT244SC, Q1 IRF9321PBF, Q10 FDN337N, Q11 FDN337N, Q12 BSS138, Q13 BSS138, Q14 FDN337N, Q2 BSS670, Q3 BSS138, Q4 BSS670, Q5 BSS138, Q6 BSS316, Q7 BSS138, Q8 BSS138, Q9 BSS670, U1 MAX202CDWR, U2 74HCT595D, U3 TC7SU04F, U4 AL8805WS, U5 AL8805WS, U6 TC7SU04F, X1 USB

Commit message: major changes : - carte pieuvre - carte relais - correctif v1 : usb + pin A7 ! - enclosure
Parts:
- removed A+_UART: (no value), SparkFun:M02LOCK_LONGPADS
- removed C20, C25, C27, C28: 0.1uF, rcl:C-EUC0603
- removed EXT2: EXT, pierre_vv:EXT-DNC
- removed F2, F3, F4, F5: PTC1812, pierre_vv:PTC1812
- removed GYRO-LED: PLUG-6, pierre_vv:M06
- removed IC1: LM2596S, national-semiconductor:LM2596S
- removed IC2: 74ACT244SC, 74xx-us:74S244DW
- removed INPUT: PLUG-8, pierre_vv:M08
- removed JP1: CHARGEUR, pierre_vv:M05X2
- removed LG, LR: (no value), SparkFun-LED:LED1206
- removed Q10, Q11, Q14: FDN337N, SparkFun-DiscreteSemi:MOSFET-NCHANNELBSS316
- removed Q12, Q13: BSS138, SparkFun-DiscreteSemi:MOSFET-NCHANNELBSS138
- removed R33, R35, R48: 20K, SparkFun-Passives:RESISTOR0603-RES
- removed R34, R36, R37, R38, R39, R40, R43, R44, R47: 10K, SparkFun-Passives:RESISTOR0603-RES
- removed R41, R42: 1K, SparkFun-Passives:RESISTOR0603-RES
- removed R49: 22K, SparkFun-Passives:RESISTOR0603-RES
- removed R50: 33K, SparkFun-Passives:RESISTOR0603-RES
- removed R51: 100K, SparkFun-Passives:RESISTOR0603-RES
- removed RAW_IN: DNC_IN2PWR, pierre_vv:DNC_IN2PWR
- removed RELAY: PLUG-3, pierre_vv:M03
- removed RELAY1: G5L, relay:G5L
- removed RGB-LED: RJ45-RGBLED, con-amphenol-rj45-ld:RJ45-RGBLED
- removed RS232: (no value), SparkFun-Connectors:M03LOCK
- removed TITREUR1, TITREUR2: DNC_TITREUR, pierre_vv:DNC_TITREUR
- removed U$8: RJ45-EXTDNC, con-amphenol-rj45-ld:RJ45-EXTDNC
- removed X1: USB, pierre_vv:USB
- added C6, C8: 1uF, rcl:C-EUC0603
- added C7, C9: 0.1uF, rcl:C-EUC0603
- added D3, D7, D8: 40v5A, pierre_vv:DIODE_SCHOTKYSMPA
- added D9: 10V, SparkFun-DiscreteSemi:DIODE-ZENERSOD-123
- added FAN1, FAN2, FAN3, FAN4, FAN5, FAN6, FAN7, FAN8, LED10W3, LED10W4, LED10W5, LED10W6, LED10W7, LED10W8, POT, SWITCH: PLUG-2, pierre_vv:M02PLUG
- added L4, L5, L6, L7, L8: 100nH2.4A, SparkFun:INDUCTORPWR
- added L9: LG, SparkFun-LED:LED1206
- added RAW_IN1: DNC_IN2PWR, pierre_vv:DNC_IN2PWR
- added SJ3, SJ4, SJ5, SJ6: JUMPER-PAD-3-2OF3_NC_BY_TRACE_LARGE, SparkFun-Passives:JUMPER-PAD-3-2OF3_NC_BY_TRACE_LARGE
- added U$3, U$5: RADIATEUR, pierre_vv:RADIATEUR
- added U7, U8: AL8805WS, SparkFun-PowerIC:AL8805
- added U9: PCA9685PW, pierre_vv:PCA9685PW
- C1, C5: value 220uF -> 0.1uF; device SparkFun:CAP_POLE -> rcl:C-EUC0603; OC_FARNELL 1800687 -> (none)
- C10: value 0.1uF -> 1uF; VMIN 50V -> (none)
- C11: VMIN (none) -> 50V
- C14: value 1uF -> 0.1uF
- C17, C18, C19: value 0.1uF -> 220uF; device rcl:C-EUC0603 -> SparkFun:CAP_POLE; OC_FARNELL (none) -> 1800687; VMIN (none) -> 50V
- C2: value 100u -> 1uF; device rcl:CPOL-USD -> rcl:C-EUC0603; OC_FARNELL 2326175RL -> (none)
- C3: value 100u -> 0.1uF; device rcl:CPOL-USD -> rcl:C-EUC0603; OC_FARNELL 2326175RL -> (none); VMIN (none) -> 50V
- C4: value 220uF -> 1uF; device SparkFun:CAP_POLE -> rcl:C-EUC0603; OC_FARNELL 1800687 -> (none); VMIN 50V -> (none)
- D2: value 10V -> 40v5A; device SparkFun-DiscreteSemi:DIODE-ZENERSOD-123 -> pierre_vv:DIODE_SCHOTKYSMPA; OC_FARNELL 1431256 -> 1861427
- D6: value (none) -> 40v5A; device SparkFun-DiscreteSemi:DIODESMA-ALT -> pierre_vv:DIODE_SCHOTKYSMPA; OC_FARNELL 2101190 -> 1861427
- L1: value 68nH3A -> 100nH2.4A; OC_FARNELL 2288510 -> 1864459RL
- Q1: value IRF9321PBF -> BSS316; device pierre_vv:IRF9321PBF -> SparkFun-DiscreteSemi:MOSFET-NCHANNELBSS316
- Q2, Q4: value BSS670 -> BSS316
- Q3, Q5, Q7, Q8: value BSS138 -> BSS316; device SparkFun-DiscreteSemi:MOSFET-NCHANNELBSS138 -> SparkFun-DiscreteSemi:MOSFET-NCHANNELBSS316
- Q9: value BSS670 -> IRF9321PBF; device SparkFun-DiscreteSemi:MOSFET-NCHANNELBSS316 -> pierre_vv:IRF9321PBF
- R1, R13, R14: value 100K -> 0.110; device SparkFun-Passives:RESISTOR0603-RES -> rcl:R-US_R0805
- R10, R11: value 33K -> OPT; device SparkFun-Passives:RESISTOR0603-RES -> rcl:R-US_R0805; MOUNT (none) -> NO
- R12: value 5.1K -> 100K
- R15, R16, R4: value 100K -> OPT; device SparkFun-Passives:RESISTOR0603-RES -> rcl:R-US_R0805; MOUNT (none) -> NO
- R2: value 100k1% -> 0.110; device SparkFun-Passives:RESISTOR0603-RES -> rcl:R-US_R0805
- R26, R32: value 100K -> 1K
- R27, R29, R30: value 100K -> 10K
- R3: value 10k1% -> OPT; device SparkFun-Passives:RESISTOR0603-RES -> rcl:R-US_R0805; MOUNT (none) -> NO
- R7, R8: value 56K -> 0.110; device SparkFun-Passives:RESISTOR0603-RES -> rcl:R-US_R0805
- SJ1, SJ2: value JUMPER-PAD-3-NO -> JUMPER-PAD-3-2OF3_NC_BY_TRACE_LARGE; device SparkFun-Passives:JUMPER-PAD-3-NO -> SparkFun-Passives:JUMPER-PAD-3-2OF3_NC_BY_TRACE_LARGE
- U$4: value RASPIA+ -> RADIATEUR; device pierre_vv:RASPIA+ -> pierre_vv:RADIATEUR; OC_FARNELL (none) -> 1703172
- U1: value MAX202CDWR -> AL8805WS; device SparkFun-DigitalIC:MAX232SOIC16 -> SparkFun-PowerIC:AL8805; OC_FARNELL 2382871 -> (none)
- U2: value 74HCT595D -> AL8805WS; device IC:74HCT595D -> SparkFun-PowerIC:AL8805; OC_FARNELL 2445164 -> (none)
- U3, U6: value TC7SU04F -> AL8805WS; device SparkFun-DigitalIC:INVERTER_SOT23-5 -> SparkFun-PowerIC:AL8805; OC_FARNELL 1105925 -> (none)
Connections:
- removed net +3V3: Q13.G, Q3.G, R38.2, R44.2, U$4.3.3V, U$4.3.3V_2
- removed net /REG_RCK_5V=ACTIVE_CS: U2.G, U6.Y
- removed net ALL_CS_ENABLE_ACTIVE_LOW_5V: IC2A.G, IC2B.G, U3.Y
- removed net ANALOG_RAW: AT328.ADC7, Q7.S, R3.2
- removed net ATMEGA_CS: IC2B.A2, U$4.GPIO13
- removed net ATMEGA_CS_5V: AT328.PB2(SS/OC1B), IC2B.Y2
- removed net CHARGING: JP1.2, U$4.GPIO23
- removed net CS_TRIGGER_ACTIVE_HIGH: R39.2, U$4.GPIO5, U3.A
- removed net DIGITAL_LED2_OR_FLEX3: AT328.PC1(ADC1), SJ1.2
- removed net EXT1_CS: IC2A.A4, U$4.GPIO2
- removed net EXT2_CS: IC2A.A3, U$4.GPIO3
- removed net EXT2_CS_5V: EXT2.CS, IC2A.Y3
- removed net EXT3_CS: IC2A.A2, U$4.GPIO4
- removed net EXT3_CS_5V: IC2A.Y2
- removed net GYRO_1: AT328.PC5(ADC5/SCL), Q4.G, R28.2
- removed net GYRO_2: AT328.PC4(ADC4/SDA), Q2.G, R27.2
- removed net GYRO_3: AT328.PC3(ADC3), Q6.G, R26.2
- removed net GYRO_4: AT328.PC2(ADC2), Q9.G, R25.2
- removed net INT_ATMEGA: R35.2, R36.1, U$4.GPIO20
- removed net INT_ATMEGA_5V: AT328.PD4(XCK/T0), R36.2
- removed net INT_TELECO: R33.2, R34.1, U$4.GPIO21
- removed net INT_TELECO_5V: R34.2, U$8.INT
- removed net LEDR: LR.C, Q8.D
- removed net LED_G: Q12.G, R31.2, U$4.GPIO16
- removed net LED_R: Q8.G, R32.2, U$4.GPIO12
- removed net LG: LG.C, Q12.D
- removed net MISO: Q3.S, R38.1, U$4.GPIO9
- removed net MOSI: IC2B.A4, U$4.GPIO10
- removed net N$1: D1.C, IC1.OUT, L1.1
- removed net N$19: F3.1, Q10.D
- removed net N$20: INPUT.6, R10.1, R7.1
- removed net N$21: LR.A, R42.1
- removed net N$23: INPUT.5, R11.1, R8.1
- removed net N$24: C19.2, U1.V+
- removed net N$26: R49.2, R50.2, X1.D+, X1.D-
- removed net N$29: F5.2, RGB-LED.R
- removed net N$50: C18.2, U1.C2-
- removed net N$51: C18.1, U1.C2+
- removed net N$52: C17.2, U1.C1-
- removed net N$53: C17.1, U1.C1+
- removed net PRXD_PIN2_RS232: RS232.1, U1.T2OUT
- removed net PTXD_PIN3_RS232: RS232.2, U1.R2IN
- removed net PUSH2: AT328.PD7(AIN1), C14.1, R10.2
- removed net PUSH3: AT328.PB0(ICP), C13.1, R11.2
- removed net PWM_FLEX_1: AT328.PD3(INT1), Q14.G, R51.2
- removed net PWM_FLEX_2: AT328.PB1(OC1A), Q10.G, R30.2
- removed net PWM_FLEX_3: Q11.G, R29.2, SJ1.3, SJ2.3
- removed net PWM_LED2_OR_FLEX3: AT328.PD6(AIN0), SJ2.2
- removed net RAW_POL_PROTECTED: D2.C, F1.1, Q1.S, TVS.2
- removed net RAW_UNPROTECTED: JP1.3, JP1.5, JP1.7, JP1.9, Q1.D, RAW_IN.+
- removed net READ_BATTERY: Q7.G, R4.2, U$4.GPIO25
- removed net REG_RCK: IC2A.A1, U$4.GPIO17
- removed net REG_RCK_5V: IC2A.Y1, R43.2, U2.RCK, U6.A
- removed net RELAY1: Q5.G, R22.2, U$4.GPIO26
- removed net RELAY_CHARGE_BOARD: JP1.1, U$4.GPIO24
- removed net RESET: Q13.S, R44.1, U$4.GPIO27
- removed net RST1: R16.1, TITREUR1.1, U2.QD
- removed net RST2: R14.1, TITREUR1.2, U2.QB
- removed net RST3: R13.1, TITREUR1.3, U2.QA
- removed net RST4: R15.1, TITREUR1.4, U2.QC
- removed net RST5: R19.1, TITREUR2.1, U2.QG
- removed net RST6: R20.1, TITREUR2.2, U2.QH
- removed net RST7: R17.1, TITREUR2.3, U2.QE
- removed net RST8: R18.1, TITREUR2.4, U2.QF
- removed net RXA+: R47.1, R48.2, U$4.GPIO15
- removed net RXA+_5V: A+_UART.2, R47.2, U1.R2OUT
- removed net SCK: IC2B.A3, U$4.GPIO11
- removed net TELECO_CS: IC2B.A1, U$4.GPIO19
- removed net TELECO_CS_5V: IC2B.Y1, U$8./CS
- removed net TXA+_5V: A+_UART.1, U$4.GPIO14, U1.T2IN
- new net A0: SJ1.2, U9.A0
- new net A1: SJ2.2, U9.A1
- new net A2: SJ3.2, U9.A2
- new net A3: SJ4.2, U9.A3
- new net A4: SJ5.2, U9.A4
- new net A5: SJ6.2, U9.A5
- new net LED: AT328.PD3(INT1), L9.A
- new net LED+3: C4.1, LED10W3.1, R2.1, R3.1, U2.SET
- new net LED+4: C2.1, LED10W4.1, R1.1, R4.1, U1.SET
- new net LED+5: C21.1, LED10W5.1, R23.1, R45.1, U5.SET
- new net LED+6: C23.1, LED10W6.1, R24.1, R46.1, U4.SET
- new net LED+7: C13.1, LED10W7.1, R14.1, R15.1, U8.SET
- new net LED+8: C10.1, LED10W8.1, R13.1, R16.1, U7.SET
- new net LED-3: C4.2, L4.2, LED10W3.2
- new net LED-4: C2.2, L1.2, LED10W4.2
- new net LED-5: C21.2, L3.2, LED10W5.2
- new net LED-6: C23.2, L2.2, LED10W6.2
- new net LED-7: C13.2, L8.2, LED10W7.2
- new net LED-8: C10.2, L7.2, LED10W8.2
- new net OE: AT328.PD4(XCK/T0), R27.1, U9.~OE
- new net PWM_FAN1: Q4.G, R28.2, U9.LED8
- new net PWM_FAN2: Q1.G, R12.2, U9.LED9
- new net PWM_FAN3: Q2.G, R17.2, U9.LED10
- new net PWM_FAN4: Q3.G, R18.2, U9.LED11
- new net PWM_FAN5: Q5.G, R19.2, U9.LED12
- new net PWM_FAN6: Q6.G, R20.2, U9.LED13
- new net PWM_FAN7: Q7.G, R22.2, U9.LED14
- new net PWM_FAN8: Q8.G, R25.2, U9.LED15
- new net PWM_LED_3: U2.CTRL, U9.LED2
- new net PWM_LED_4: U1.CTRL, U9.LED3
- new net PWM_LED_5: U5.CTRL, U9.LED4
- new net PWM_LED_6: U4.CTRL, U9.LED5
- new net PWM_LED_7: U8.CTRL, U9.LED6
- new net PWM_LED_8: U7.CTRL, U9.LED7
- new net RAW_POL_PROTECTED1: D9.C, F1.1, Q9.S, TVS.2
- new net RAW_UNPROTECTED1: Q9.D, RAW_IN1.+
- new net SCL: AT328.PC5(ADC5/SCL), R29.1, U9.SCL
- new net SDA: AT328.PC4(ADC4/SDA), R30.1, U9.SDA
- net +5V: now also C14.1, R26.2, R27.2, R29.2, R30.2, U9.VDD; no longer C11.1, C19.1, C2.+, C25.1, C27.1, C28.1, C3.+, D6.C, EXT2.5V, IC1.FB, IC2P.VCC, L1.2, R13.2, R14.2, R15.2, R16.2, R17.2, R18.2, R19.2, R20.2, R37.2, R41.2, R42.2, R50.1, R7.2, R8.2, RELAY11.2, TITREUR1.12, TITREUR1.14, TITREUR1.16, TITREUR2.12, TITREUR2.14, TITREUR2.16, U$4.5V_1, U$4.5V_2, U$8.5V, U1.VCC, U2.SCL, U2.VCC, U3.VCC, U6.VCC, X1.V+
- net CODE: no longer AT328.PC0(ADC0), EXT2.COD, R12.1, U$8.COD
- net EXT1_CS_5V: now also AT328.PB2(SS/OC1B); no longer IC2A.Y4
- net FLOAT1: now also POT.2; no longer INPUT.2
- net GND: now also C1.2, C17.-, C18.-, C19.-, C3.2, C5.2, C7.2, C9.2, Q1.S, Q3.S, Q7.S, R12.1, R17.1, R18.1, R19.1, R20.1, R31.2, R32.2, RAW_IN1.-, SJ1.1, SJ2.1, SJ3.1, SJ4.1, SJ5.1, SJ6.1, SWITCH.2, U7.GND, U8.GND, U9.EXTCLK, U9.VSS; no longer C1.-, C10.2, C13.2, C2.-, C20.2, C25.2, C27.2, C28.2, C3.-, C4.-, C5.-, D1.A, EXT2.GND, IC1.!ON!/OFF, IC1.GND, IC2P.GND, INPUT.4, INPUT.8, JP1.10, JP1.4, JP1.6, JP1.8, Q10.S, Q11.S, Q12.S, Q14.S, Q9.S, R1.2, R12.2, R26.1, R27.1, R29.1, R3.1, R30.1, R31.1, R32.1, R33.1, R35.1, R39.1, R4.1, R40.1, R43.1, R48.1, R49.1, R51.1, RAW_IN.-, RS232.3, TITREUR1.11, TITREUR1.13, TITREUR1.15, TITREUR1.8, TITREUR2.11, TITREUR2.13, TITREUR2.15, TITREUR2.8, U$4.GND, U$4.GND_2, U$4.GND_3, U$4.GND_4, U$4.GND_5, U$4.GND_6, U$4.GND_7, U$4.GND_8, U$8.GND, X1.GND
- net LED+1: now also C6.1, R11.1, R7.1, U3.SET; no longer C23.1, R24.1, R46.1, U4.SET
- net LED+2: now also C8.1, R10.1, R8.1, U6.SET; no longer C21.1, R23.1, R45.1, U5.SET
- net LED-1: now also C6.2, L5.2; no longer C23.2, L2.2
- net LED-2: now also C8.2, L6.2; no longer C21.2, L3.2
- net MISO_5V: no longer EXT2.MISO, Q3.D, R37.1, U$8.MISO
- net MOSI_5V: no longer EXT2.MOSI, IC2B.Y4, TITREUR1.7, TITREUR2.7, U$8.MOSI, U2.SER
- net N$10: now also D7.A, L7.1, U7.SW; no longer GYRO-LED.2, Q4.D
- net N$11: now also D8.A, L8.1, U8.SW; no longer GYRO-LED.3, Q2.D
- net N$12: now also FAN2.1, Q1.D; no longer GYRO-LED.4, Q6.D
- net N$13: now also FAN3.1, Q2.D; no longer GYRO-LED.5, Q9.D
- net N$14: now also FAN4.1, Q3.D; no longer F4.2, RGB-LED.B
- net N$15: now also FAN5.1, Q5.D; no longer RELAY.3, RELAY12.O
- net N$16: now also FAN6.1, Q6.D; no longer D6.A, Q5.D, RELAY11.1
- net N$17: now also FAN7.1, Q7.D; no longer F4.1, Q11.D
- net N$18: now also FAN8.1, Q8.D; no longer LG.A, R41.1
- net N$22: now also SWITCH.1; no longer INPUT.7
- net N$25: now also POT.1; no longer INPUT.1
- net N$3: now also D1.A, L1.1, U1.SW; no longer Q7.D, R2.1
- net N$30: now also R26.1, SJ1.3, SJ2.3, SJ3.3, SJ4.3, SJ5.3, SJ6.3; no longer F5.1, Q14.D
- net N$35: now also L9.C, R32.1; no longer C20.1, U1.V-
- net N$4: now also FAN1.1, Q4.D; no longer RELAY.1, RELAY12.S
- net N$5: now also D2.A, L4.1, U2.SW; no longer F2.2, GYRO-LED.1, GYRO-LED.6
- net N$8: now also D3.A, L5.1, U3.SW; no longer RELAY.2, RELAY12.P
- net N$9: now also D6.A, L6.1, U6.SW; no longer F3.2, RGB-LED.G
- net PROTECT_GATE: now also D9.A, Q9.G, R31.1; no longer D2.A, Q1.G, R1.1
- net PWM_LED_1: now also U6.CTRL, U9.LED0; no longer AT328.PD5(T1), U5.CTRL
- net PWM_LED_2: now also U3.CTRL, U9.LED1; no longer SJ1.1, SJ2.1, U4.CTRL
- net RAW_FUSED: now also C1.1, C11.1, C17.+, C18.+, C19.+, C3.1, C5.1, C7.1, C9.1, D1.C, D2.C, D3.C, D6.C, D7.C, D8.C, FAN1.2, FAN2.2, FAN3.2, FAN4.2, FAN5.2, FAN6.2, FAN7.2, FAN8.2, R1.2, R10.2, R11.2, R13.2, R14.2, R15.2, R16.2, R3.2, R4.2, R7.2, R8.2, U1.VIN, U2.VIN, U3.VIN, U6.VIN, U7.VIN, U8.VIN; no longer C1.+, C10.1, C4.+, C5.+, EXT1.RAW, EXT2.RAW, F2.1, IC1.VIN, RGB-LED.VCC
- net RESET_5V: no longer Q13.D
- net SCK_5V: no longer EXT2.SCK, IC2B.Y3, R40.2, TITREUR1.5, TITREUR2.5, U$8.SCK, U2.SCK
Other:
- note removed: "2x FLEX DRIVER"
- note removed: "4x FLEX GYRO on/off DRIVER"
- note removed: "5V buck converter and 3.3V LDO"
- note removed: "CS titreur driver"
- note removed: "LEDS"
- note removed: "LEVEL SHIFT 3.3V TO 5V"
- note removed: "RELAY"
- note removed: "RPI DOCK"
- note removed: "RS232"
- note removed: "attention - analog_raw et digital _ledorflex interverti pour la prochaine version"
- note removed: "reverse + overvoltage protection"
- moved on the sheet: 16MHZ, AT328, C10, C11, C12, C13, C14, C15, C16, C21, C22, C23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
